File: Amplificateur_Audio/Amplificateur_Audio_Avant_Projet/Amplificateur_Audio.kicad_sch (KiCad schematic)
At the start: 0 parts

Commit message: Correction du nom de l'entreprise
Other:
- company: NDG -> NDH
Changed lines of the file:
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@@
 		(date "2025-05-19")
 		(rev "1.0")
-		(company "NDG")
+		(company "NDH")
 	)
 	(sheet
