File: Amplificateur_Audio/Amplificateur_Audio_Avant_Projet/Analog_Io_Board.kicad_sch (KiCad schematic)
At the start: 147 parts, among them J1101 SURROUND-LEFT, J1102 UPMIX-LEFT, J1103 FR-TWEETER, J1104 FL-TWEETER, J1105 CENTER-TWEETER, J1106 SURROUND-RIGHT, J1107 UPMIX-RIGHT, J1108 FR-WOOFER, J1109 FL-WOOFER, J1110 CENTER-WOOFER, J1111 Analog OUTPUT Connector, U1101 NE5532AD, U1102 NE5532AD, U1103 NE5532AD, U1104 NE5532AD, U1105 NE5532AD, U1106 NE5532AD, U1107 NE5532AD, U1108 NE5532AD, U1109 NE5532AD, U1110 NE5532AD

Commit message: Correction du nom de l'entreprise
Other:
- company: NDG -> NDH
Changed lines of the file:
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@@
 		(date "2025-05-19")
 		(rev "1.0")
-		(company "NDG")
+		(company "NDH")
 	)
 	(rectangle
