File: Amplificateur_Audio/Amplificateur_Audio_Avant_Projet/Center_Channel.kicad_sch (KiCad schematic)
At the start: 78 parts, among them J801 Center Tweeter+, J802 Center Tweeter-, J803 Center Woofer+, J804 Center Woofer-, U801 PCM5252RHBR, U802 TPA3244DDWR

Commit message: Correction du nom de l'entreprise
Other:
- company: NDG -> NDH
Changed lines of the file:
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@@
 		(date "2025-05-19")
 		(rev "1.0")
-		(company "NDG")
+		(company "NDH")
 	)
 	(rectangle
