File: Amplificateur_Audio/Amplificateur_Audio_Avant_Projet/Clock_Drivers.kicad_sch (KiCad schematic)
At the start: 59 parts, among them J301 Conn_02x10_Odd_Even, Q301 NMOS, Q302 NMOS, U301 74LVC1G125, U302 74LVC1G125, U303 74LVC1G125, U304 74LVC1G125, U305 74LVC1G125, U306 74LVC1G125, U307 74LVC1G125, U308 74LVC1G125, U309 74LVC1G125, U310 74LVC1G125

Commit message: Correction du nom de l'entreprise
Other:
- company: NDG -> NDH
Changed lines of the file:
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@@
 		(date "2025-05-19")
 		(rev "1.0")
-		(company "NDG")
+		(company "NDH")
 	)
 	(rectangle
