File: Amplificateur_Audio/Amplificateur_Audio_Avant_Projet/Front_Right_Channel.kicad_sch (KiCad schematic)
At the start: 78 parts, among them J601 Front Right Tweeter+, J602 Front Right Tweeter-, J603 Front Right Woofer+, J604 Front Right Woofer-, U601 PCM5252RHBR, U602 TPA3244DDWR

Commit message: Correction du nom de l'entreprise
Other:
- company: NDG -> NDH
Changed lines of the file:
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@@
 		(date "2025-05-19")
 		(rev "1.0")
-		(company "NDG")
+		(company "NDH")
 	)
 	(rectangle
