File: Amplificateur_Audio/Amplificateur_Audio_Avant_Projet/MSP54_IO.kicad_sch (KiCad schematic)
At the start: 97 parts, among them J201 JTAG, J202 Conn_01x02, J203 Conn_02x08_Odd_Even, Q201 NPN, Q202 NPN, Q203 NPN, Q204 NPN, Q205 NPN, Q206 NPN, SW201 MUTE, SW202 VOL+, SW203 VOL-, SW204 MODE1, SW205 MODE2, SW206 MODE3, SW207 MODE4, SW208 LOAD, SW209 RESET, U201 MSP430F5234IRGZ, U202 TCA6408ARSVR, U203 24LC512, U204 TCA9548ARGER, Y201 32.768kHz

Commit message: Correction du nom de l'entreprise
Other:
- company: NDG -> NDH
Changed lines of the file:
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@@
 		(date "2025-05-19")
 		(rev "1.0")
-		(company "NDG")
+		(company "NDH")
 	)
 	(rectangle
