File: Amplificateur_Audio/Amplificateur_Audio_Avant_Projet/Surrond_Channel.kicad_sch (KiCad schematic)
At the start: 84 parts, among them J401 Surrond Left+, J405 Analog input Connector, U401 PCM5252RHBR, U402 TPA3244DDWR, U403 74LVC1G125, U404 74LVC1G125

Commit message: Correction du nom de l'entreprise
Other:
- company: NDG -> NDH
Changed lines of the file:
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@@
 		(date "2025-05-19")
 		(rev "1.0")
-		(company "NDG")
+		(company "NDH")
 	)
 	(rectangle
