File: Amplificateur_Audio/Amplificateur_Audio_Avant_Projet/Up_Channel.kicad_sch (KiCad schematic)
At the start: 78 parts, among them J502 UP LEFT+, J503 UP LEFT-, J504 UP RIGHT+, J505 UP RIGHT-, U501 PCM5252RHBR, U502 TPA3244DDWR

Commit message: Correction du nom de l'entreprise
Other:
- company: NDG -> NDH
Changed lines of the file:
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@@
 		(date "2025-05-19")
 		(rev "1.0")
-		(company "NDG")
+		(company "NDH")
 	)
 	(rectangle
