File: Amplificateur_Audio/Amplificateur_Audio_Custom/Amplificateur_Audio.kicad_pcb (KiCad board)
At the start: 2 copper layers, 0 parts

Commit message: Ajout de point de test et début du routage
Parts:
- added C1001: 47uF, Capacitor_SMD:CP_Elec_8x6.2, F.Cu at (119.6, 209.3)
- added C1002: 1uF, Capacitor_SMD:C_0603_1608Metric_Pad1.08x0.95mm_HandSolder, F.Cu at (391.2, 145.3)
- added C1003: 0.01uF, Capacitor_SMD:C_0603_1608Metric_Pad1.08x0.95mm_HandSolder, F.Cu at (391.2, 151.3)
- added C1004: 0.1uF, Capacitor_SMD:C_0603_1608Metric_Pad1.08x0.95mm_HandSolder, F.Cu at (12.6, 141.3)
- added C1005: 2.2uF, Capacitor_SMD:C_0805_2012Metric_Pad1.18x1.45mm_HandSolder, F.Cu at (391.2, 148.3)
- added C1006: 2.2uF, Capacitor_SMD:C_0805_2012Metric_Pad1.18x1.45mm_HandSolder, F.Cu at (391.2, 154.3)
- added C1007: 3600pF, Capacitor_SMD:C_0603_1608Metric_Pad1.08x0.95mm_HandSolder, F.Cu at (17.6, 129.3)
- added C1008: 75pF, Capacitor_SMD:C_0603_1608Metric_Pad1.08x0.95mm_HandSolder, F.Cu at (17.6, 132.3)
- added C1009: 47uF, Capacitor_SMD:CP_Elec_8x6.2, F.Cu at (441.5, 249.1)
- added C1010: 2.2uF, Capacitor_SMD:C_0805_2012Metric_Pad1.18x1.45mm_HandSolder, F.Cu at (272.0, 176.0)
- added C1011: 0.47uF, Capacitor_SMD:C_0603_1608Metric_Pad1.08x0.95mm_HandSolder, F.Cu at (272.0, 173.0)
- added C1012: 4.7uF, Capacitor_SMD:C_1206_3216Metric_Pad1.33x1.80mm_HandSolder, F.Cu at (442.5, 207.1)
- added C1013: 47uF, Capacitor_SMD:CP_Elec_6.3x5.8, F.Cu at (440.5, 258.1)
- added C1014: 0.1uF, Capacitor_SMD:C_0603_1608Metric_Pad1.08x0.95mm_HandSolder, F.Cu at (277.0, 169.0)
- added C1015: 10uF, Capacitor_SMD:CP_Elec_6.3x5.8, F.Cu at (440.5, 267.1)
- added C1016: 100uF, Capacitor_SMD:CP_Elec_6.3x5.8, F.Cu at (464.5, 260.1)
- added C1017: 4.7uF, Capacitor_SMD:C_1206_3216Metric_Pad1.33x1.80mm_HandSolder, F.Cu at (442.5, 204.1)
- added C1018: 0.47uF, Capacitor_SMD:C_0603_1608Metric_Pad1.08x0.95mm_HandSolder, F.Cu at (272.0, 170.0)
- added C1019: 47uF, Capacitor_SMD:CP_Elec_6.3x5.8, F.Cu at (454.5, 200.1)
- added C1020: 0.1uF, Capacitor_SMD:C_0603_1608Metric_Pad1.08x0.95mm_HandSolder, F.Cu at (183.9, 129.2)
- added C1021: 10uF, Capacitor_SMD:CP_Elec_6.3x5.8, F.Cu at (454.5, 186.1)
- added C1022: 100uF, Capacitor_SMD:CP_Elec_6.3x5.8, F.Cu at (36.6, 231.3)
- added C1023: 10uF, Capacitor_SMD:CP_Elec_6.3x5.8, F.Cu at (452.5, 175.1)
- added C1024: 100uF, Capacitor_SMD:CP_Elec_6.3x5.8, F.Cu at (129.6, 191.3)
- added C1101: 0.1uF, Capacitor_SMD:C_0402_1005Metric_Pad0.74x0.62mm_HandSolder, F.Cu at (42.6, 220.3)
- added C1102: 10uF, Capacitor_SMD:C_1206_3216Metric_Pad1.33x1.80mm_HandSolder, F.Cu at (83.6, 190.3)
- added C1103: 22pF, Capacitor_SMD:C_0603_1608Metric_Pad1.08x0.95mm_HandSolder, F.Cu at (72.6, 245.3)
- added C1104: 22pF, Capacitor_SMD:C_0603_1608Metric_Pad1.08x0.95mm_HandSolder, F.Cu at (68.6, 241.3)
- added C1105: 10uF, Capacitor_SMD:C_1206_3216Metric_Pad1.33x1.80mm_HandSolder, F.Cu at (67.6, 238.3)
- added C1106: 0.1uF, Capacitor_SMD:C_0402_1005Metric_Pad0.74x0.62mm_HandSolder, F.Cu at (85.6, 209.3)
- added C1107: 22pF, Capacitor_SMD:C_0603_1608Metric_Pad1.08x0.95mm_HandSolder, F.Cu at (78.6, 159.3)
- added C1108: 22pF, Capacitor_SMD:C_0603_1608Metric_Pad1.08x0.95mm_HandSolder, F.Cu at (78.6, 172.3)
- added C1109: 10uF, Capacitor_SMD:C_1206_3216Metric_Pad1.33x1.80mm_HandSolder, F.Cu at (83.6, 193.3)
- added C1110: 0.1uF, Capacitor_SMD:C_0402_1005Metric_Pad0.74x0.62mm_HandSolder, F.Cu at (82.6, 217.3)
- added C1111: 22pF, Capacitor_SMD:C_0603_1608Metric_Pad1.08x0.95mm_HandSolder, F.Cu at (77.6, 192.3)
- added C1112: 22pF, Capacitor_SMD:C_0603_1608Metric_Pad1.08x0.95mm_HandSolder, F.Cu at (89.6, 237.3)
- added C1113: 10uF, Capacitor_SMD:C_1206_3216Metric_Pad1.33x1.80mm_HandSolder, F.Cu at (110.6, 234.3)
- added C1114: 0.1uF, Capacitor_SMD:C_0402_1005Metric_Pad0.74x0.62mm_HandSolder, F.Cu at (85.6, 217.3)
- added C1115: 22pF, Capacitor_SMD:C_0603_1608Metric_Pad1.08x0.95mm_HandSolder, F.Cu at (83.6, 262.3)
- added C1116: 22pF, Capacitor_SMD:C_0603_1608Metric_Pad1.08x0.95mm_HandSolder, F.Cu at (67.6, 247.3)
- added C1117: 10uF, Capacitor_SMD:C_1206_3216Metric_Pad1.33x1.80mm_HandSolder, F.Cu at (113.6, 215.3)
- added C1118: 0.1uF, Capacitor_SMD:C_0402_1005Metric_Pad0.74x0.62mm_HandSolder, F.Cu at (46.6, 220.3)
- added C1119: 22pF, Capacitor_SMD:C_0603_1608Metric_Pad1.08x0.95mm_HandSolder, F.Cu at (67.6, 244.3)
- added C1120: 22pF, Capacitor_SMD:C_0603_1608Metric_Pad1.08x0.95mm_HandSolder, F.Cu at (72.6, 248.3)
- added C1121: 10uF, Capacitor_SMD:C_1206_3216Metric_Pad1.33x1.80mm_HandSolder, F.Cu at (74.6, 229.3)
- added C1122: 0.1uF, Capacitor_SMD:C_0402_1005Metric_Pad0.74x0.62mm_HandSolder, F.Cu at (110.6, 256.3)
- added C1123: 22pF, Capacitor_SMD:C_0603_1608Metric_Pad1.08x0.95mm_HandSolder, F.Cu at (112.6, 179.3)
- added C1124: 22pF, Capacitor_SMD:C_0603_1608Metric_Pad1.08x0.95mm_HandSolder, F.Cu at (123.6, 225.3)
- added C1125: 10uF, Capacitor_SMD:C_1206_3216Metric_Pad1.33x1.80mm_HandSolder, F.Cu at (109.6, 212.3)
- added C1126: 0.1uF, Capacitor_SMD:C_0402_1005Metric_Pad0.74x0.62mm_HandSolder, F.Cu at (115.6, 230.3)
- added C1127: 22pF, Capacitor_SMD:C_0603_1608Metric_Pad1.08x0.95mm_HandSolder, F.Cu at (100.6, 169.3)
- added C1128: 22pF, Capacitor_SMD:C_0603_1608Metric_Pad1.08x0.95mm_HandSolder, F.Cu at (114.6, 182.3)
- added C1129: 10uF, Capacitor_SMD:C_1206_3216Metric_Pad1.33x1.80mm_HandSolder, F.Cu at (103.6, 232.3)
- added C1130: 0.1uF, Capacitor_SMD:C_0402_1005Metric_Pad0.74x0.62mm_HandSolder, F.Cu at (107.6, 200.3)
- added C1131: 22pF, Capacitor_SMD:C_0603_1608Metric_Pad1.08x0.95mm_HandSolder, F.Cu at (107.6, 161.3)
- added C1132: 22pF, Capacitor_SMD:C_0603_1608Metric_Pad1.08x0.95mm_HandSolder, F.Cu at (107.6, 185.3)
- added C1133: 10uF, Capacitor_SMD:C_1206_3216Metric_Pad1.33x1.80mm_HandSolder, F.Cu at (103.6, 181.3)
- added C1134: 0.1uF, Capacitor_SMD:C_0402_1005Metric_Pad0.74x0.62mm_HandSolder, F.Cu at (118.6, 230.3)
- added C1135: 22pF, Capacitor_SMD:C_0603_1608Metric_Pad1.08x0.95mm_HandSolder, F.Cu at (83.6, 265.3)
- added C1136: 22pF, Capacitor_SMD:C_0603_1608Metric_Pad1.08x0.95mm_HandSolder, F.Cu at (114.6, 272.3)
- added C1137: 10uF, Capacitor_SMD:C_1206_3216Metric_Pad1.33x1.80mm_HandSolder, F.Cu at (117.6, 225.3)
- added C1138: 0.1uF, Capacitor_SMD:C_0402_1005Metric_Pad0.74x0.62mm_HandSolder, F.Cu at (104.6, 203.3)
- added C1139: 22pF, Capacitor_SMD:C_0603_1608Metric_Pad1.08x0.95mm_HandSolder, F.Cu at (62.6, 244.3)
- added C1140: 22pF, Capacitor_SMD:C_0603_1608Metric_Pad1.08x0.95mm_HandSolder, F.Cu at (113.6, 164.3)
- added C1141: 10uF, Capacitor_SMD:C_0603_1608Metric_Pad1.08x0.95mm_HandSolder, F.Cu at (102.6, 166.3)
- added C1142: 0.1uF, Capacitor_SMD:C_0402_1005Metric_Pad0.74x0.62mm_HandSolder, F.Cu at (102.6, 159.3)
- added C1143: 10uF, Capacitor_SMD:C_0603_1608Metric_Pad1.08x0.95mm_HandSolder, F.Cu at (102.6, 172.3)
- added C1144: 0.1uF, Capacitor_SMD:C_0402_1005Metric_Pad0.74x0.62mm_HandSolder, F.Cu at (102.6, 149.3)
- added C1145: 10uF, Capacitor_SMD:C_0603_1608Metric_Pad1.08x0.95mm_HandSolder, F.Cu at (102.6, 175.3)
- added C1146: 0.1uF, Capacitor_SMD:C_0402_1005Metric_Pad0.74x0.62mm_HandSolder, F.Cu at (102.6, 157.3)
- added C1147: 10uF, Capacitor_SMD:C_0603_1608Metric_Pad1.08x0.95mm_HandSolder, F.Cu at (103.6, 212.3)
- added C1148: 0.1uF, Capacitor_SMD:C_0402_1005Metric_Pad0.74x0.62mm_HandSolder, F.Cu at (63.6, 216.3)
- added C1149: 10uF, Capacitor_SMD:C_0603_1608Metric_Pad1.08x0.95mm_HandSolder, F.Cu at (116.6, 228.3)
- added C1150: 0.1uF, Capacitor_SMD:C_0402_1005Metric_Pad0.74x0.62mm_HandSolder, F.Cu at (102.6, 161.3)
- added C1151: 10uF, Capacitor_SMD:C_0603_1608Metric_Pad1.08x0.95mm_HandSolder, F.Cu at (60.6, 229.3)
- added C1152: 0.1uF, Capacitor_SMD:C_0402_1005Metric_Pad0.74x0.62mm_HandSolder, F.Cu at (102.6, 147.3)
- added C1153: 10uF, Capacitor_SMD:C_0603_1608Metric_Pad1.08x0.95mm_HandSolder, F.Cu at (102.6, 178.3)
- added C1154: 0.1uF, Capacitor_SMD:C_0402_1005Metric_Pad0.74x0.62mm_HandSolder, F.Cu at (102.6, 155.3)
- added C1155: 10uF, Capacitor_SMD:C_0603_1608Metric_Pad1.08x0.95mm_HandSolder, F.Cu at (111.6, 225.3)
- added C1156: 0.1uF, Capacitor_SMD:C_0402_1005Metric_Pad0.74x0.62mm_HandSolder, F.Cu at (60.6, 216.3)
- added C1157: 10uF, Capacitor_SMD:C_0603_1608Metric_Pad1.08x0.95mm_HandSolder, F.Cu at (107.6, 215.3)
- added C1158: 0.1uF, Capacitor_SMD:C_0402_1005Metric_Pad0.74x0.62mm_HandSolder, F.Cu at (102.6, 151.3)
- added C1159: 10uF, Capacitor_SMD:C_0603_1608Metric_Pad1.08x0.95mm_HandSolder, F.Cu at (108.6, 202.3)
- added C1160: 0.1uF, Capacitor_SMD:C_0402_1005Metric_Pad0.74x0.62mm_HandSolder, F.Cu at (102.6, 153.3)
- added C1161: 10uF, Capacitor_SMD:C_0805_2012Metric_Pad1.18x1.45mm_HandSolder, F.Cu at (102.6, 215.3)
- added C1162: 10uF, Capacitor_SMD:C_0805_2012Metric_Pad1.18x1.45mm_HandSolder, F.Cu at (103.6, 201.3)
- added C1163: 0.1uF, Capacitor_SMD:C_0603_1608Metric_Pad1.08x0.95mm_HandSolder, F.Cu at (102.6, 163.3)
- added C1164: 10uF, Capacitor_SMD:C_0603_1608Metric_Pad1.08x0.95mm_HandSolder, F.Cu at (43.6, 218.3)
- added C1165: 10uF, Capacitor_SMD:C_0603_1608Metric_Pad1.08x0.95mm_HandSolder, F.Cu at (48.6, 218.3)
- added C1166: 10uF, Capacitor_SMD:C_0603_1608Metric_Pad1.08x0.95mm_HandSolder, F.Cu at (111.6, 231.3)
- added C1167: 10uF, Capacitor_SMD:C_0603_1608Metric_Pad1.08x0.95mm_HandSolder, F.Cu at (111.6, 228.3)
- added C201: 470pF, Capacitor_SMD:C_0402_1005Metric_Pad0.74x0.62mm_HandSolder, F.Cu at (150.6, 272.3)
- added C202: 470pF, Capacitor_SMD:C_0402_1005Metric_Pad0.74x0.62mm_HandSolder, F.Cu at (30.6, 219.3)
- added C203: 470pF, Capacitor_SMD:C_0402_1005Metric_Pad0.74x0.62mm_HandSolder, F.Cu at (244.4, 240.0)
- added C204: 470pF, Capacitor_SMD:C_0402_1005Metric_Pad0.74x0.62mm_HandSolder, F.Cu at (149.6, 280.3)
- added C205: 470pF, Capacitor_SMD:C_0402_1005Metric_Pad0.74x0.62mm_HandSolder, F.Cu at (136.6, 275.3)
- added C206: 470pF, Capacitor_SMD:C_0402_1005Metric_Pad0.74x0.62mm_HandSolder, F.Cu at (447.5, 264.1)
- added C207: 470pF, Capacitor_SMD:C_0402_1005Metric_Pad0.74x0.62mm_HandSolder, F.Cu at (150.6, 270.3)
- added C208: 470pF, Capacitor_SMD:C_0402_1005Metric_Pad0.74x0.62mm_HandSolder, F.Cu at (110.6, 265.3)
- added C209: 1uF, Capacitor_SMD:C_0402_1005Metric_Pad0.74x0.62mm_HandSolder, F.Cu at (224.4, 189.0)
- added C210: 0.1uF, Capacitor_SMD:C_0402_1005Metric_Pad0.74x0.62mm_HandSolder, F.Cu at (221.4, 189.0)
- added C211: 0.1uF, Capacitor_SMD:C_0402_1005Metric_Pad0.74x0.62mm_HandSolder, F.Cu at (132.6, 249.3)
- added C212: 0.1uF, Capacitor_SMD:C_0402_1005Metric_Pad0.74x0.62mm_HandSolder, F.Cu at (84.6, 274.3)
- added C213: 0.1uF, Capacitor_SMD:C_0402_1005Metric_Pad0.74x0.62mm_HandSolder, F.Cu at (450.5, 192.1)
- added C214: 0.1uF, Capacitor_SMD:C_0402_1005Metric_Pad0.74x0.62mm_HandSolder, F.Cu at (132.6, 262.3)
- added C215: 0.1uF, Capacitor_SMD:C_0402_1005Metric_Pad0.74x0.62mm_HandSolder, F.Cu at (79.6, 155.3)
- added C216: 0.1uF, Capacitor_SMD:C_0402_1005Metric_Pad0.74x0.62mm_HandSolder, F.Cu at (244.4, 216.0)
- added C217: 2200pF, Capacitor_SMD:C_0201_0603Metric_Pad0.64x0.40mm_HandSolder, F.Cu at (272.0, 147.0)
- added C218: 2200pF, Capacitor_SMD:C_0201_0603Metric_Pad0.64x0.40mm_HandSolder, F.Cu at (386.2, 161.3)
- added C219: 12pF, Capacitor_SMD:C_0402_1005Metric_Pad0.74x0.62mm_HandSolder, F.Cu at (43.6, 234.3)
- added C220: 12pF, Capacitor_SMD:C_0402_1005Metric_Pad0.74x0.62mm_HandSolder, F.Cu at (43.6, 232.3)
- added C301: 1uF, Capacitor_SMD:C_0402_1005Metric_Pad0.74x0.62mm_HandSolder, F.Cu at (131.6, 252.3)
- added C302: 0.1uF, Capacitor_SMD:C_0402_1005Metric_Pad0.74x0.62mm_HandSolder, F.Cu at (227.4, 187.0)
- added C303: 0.1uF, Capacitor_SMD:C_0402_1005Metric_Pad0.74x0.62mm_HandSolder, F.Cu at (84.6, 278.3)
- added C304: 0.1uF, Capacitor_SMD:C_0402_1005Metric_Pad0.74x0.62mm_HandSolder, F.Cu at (84.6, 272.3)
- added C305: 0.1uF, Capacitor_SMD:C_0402_1005Metric_Pad0.74x0.62mm_HandSolder, F.Cu at (226.4, 184.0)
- added C306: 0.1uF, Capacitor_SMD:C_0402_1005Metric_Pad0.74x0.62mm_HandSolder, F.Cu at (84.6, 276.3)
- added C307: 0.1uF, Capacitor_SMD:C_0402_1005Metric_Pad0.74x0.62mm_HandSolder, F.Cu at (84.6, 280.3)
- added C308: 0.1uF, Capacitor_SMD:C_0402_1005Metric_Pad0.74x0.62mm_HandSolder, F.Cu at (227.4, 189.0)
- added C401: 10uF, Capacitor_SMD:C_0603_1608Metric_Pad1.08x0.95mm_HandSolder, F.Cu at (222.5, 562.4)
- added C402: 0.1uF, Capacitor_SMD:C_0402_1005Metric_Pad0.74x0.62mm_HandSolder, F.Cu at (278.5, 533.4)
- added C403: 10uF, Capacitor_SMD:C_0603_1608Metric_Pad1.08x0.95mm_HandSolder, F.Cu at (222.5, 568.4)
- added C404: 0.1uF, Capacitor_SMD:C_0402_1005Metric_Pad0.74x0.62mm_HandSolder, F.Cu at (470.6, 496.1)
- added C405: 10uF, Capacitor_SMD:C_0603_1608Metric_Pad1.08x0.95mm_HandSolder, F.Cu at (470.6, 494.1)
- added C406: 0.1uF, Capacitor_SMD:C_0402_1005Metric_Pad0.74x0.62mm_HandSolder, F.Cu at (278.5, 537.4)
- added C407: 2.2uF, Capacitor_SMD:C_0402_1005Metric_Pad0.74x0.62mm_HandSolder, F.Cu at (438.0, 503.5)
- added C408: 2.2uF, Capacitor_SMD:C_0402_1005Metric_Pad0.74x0.62mm_HandSolder, F.Cu at (433.0, 499.5)
- added C409: 0.1uF, Capacitor_SMD:C_0402_1005Metric_Pad0.74x0.62mm_HandSolder, F.Cu at (433.0, 495.5)
- added C410: 1000pF, Capacitor_SMD:C_0402_1005Metric_Pad0.74x0.62mm_HandSolder, F.Cu at (237.5, 494.4)
- added C411: 1000pF, Capacitor_SMD:C_0402_1005Metric_Pad0.74x0.62mm_HandSolder, F.Cu at (240.5, 545.4)
- added C412: 10uF, Capacitor_SMD:C_1206_3216Metric_Pad1.33x1.80mm_HandSolder, F.Cu at (288.7, 432.9)
- added C413: 100pF, Capacitor_SMD:C_0603_1608Metric_Pad1.08x0.95mm_HandSolder, F.Cu at (282.6, 436.9)
- added C414: 10uF, Capacitor_SMD:C_1206_3216Metric_Pad1.33x1.80mm_HandSolder, F.Cu at (275.5, 433.3)
- added C415: 100pF, Capacitor_SMD:C_0603_1608Metric_Pad1.08x0.95mm_HandSolder, F.Cu at (270.2, 436.3)
- added C416: 10uF, Capacitor_SMD:C_1206_3216Metric_Pad1.33x1.80mm_HandSolder, F.Cu at (243.7, 430.6)
- added C417: 100pF, Capacitor_SMD:C_0603_1608Metric_Pad1.08x0.95mm_HandSolder, F.Cu at (249.4, 433.5)
- added C418: 10uF, Capacitor_SMD:C_1206_3216Metric_Pad1.33x1.80mm_HandSolder, F.Cu at (230.5, 432.2)
- added C419: 100pF, Capacitor_SMD:C_0603_1608Metric_Pad1.08x0.95mm_HandSolder, F.Cu at (236.1, 435.8)
- added C420: 1uF, Capacitor_SMD:C_1206_3216Metric_Pad1.33x1.80mm_HandSolder, F.Cu at (254.0, 383.6)
- added C421: 1uF, Capacitor_SMD:C_1206_3216Metric_Pad1.33x1.80mm_HandSolder, F.Cu at (260.6, 383.4)
- added C422: 1000uF, Capacitor_SMD:CP_Elec_16x17.5, F.Cu at (237.2, 364.2)
- added C423: 1uF, Capacitor_SMD:C_1206_3216Metric_Pad1.33x1.80mm_HandSolder, F.Cu at (267.1, 383.3)
- added C424: 1uF, Capacitor_SMD:C_1206_3216Metric_Pad1.33x1.80mm_HandSolder, F.Cu at (273.9, 383.2)
- added C425: 1000uF, Capacitor_SMD:CP_Elec_16x17.5, F.Cu at (267.4, 364.3)
- added C426: 0.1uF, Capacitor_SMD:C_0603_1608Metric_Pad1.08x0.95mm_HandSolder, F.Cu at (272.6, 408.4)
- added C427: 0.1uF, Capacitor_SMD:C_0603_1608Metric_Pad1.08x0.95mm_HandSolder, F.Cu at (248.0, 408.2)
- added C428: 0.1uF, Capacitor_SMD:C_0603_1608Metric_Pad1.08x0.95mm_HandSolder, F.Cu at (272.0, 412.5)
- added C429: 1uF, Capacitor_SMD:C_0603_1608Metric_Pad1.08x0.95mm_HandSolder, F.Cu at (262.7, 418.8)
- added C430: 1uF, Capacitor_SMD:C_0603_1608Metric_Pad1.08x0.95mm_HandSolder, F.Cu at (261.5, 422.8)
- added C431: 0.047uF, Capacitor_SMD:C_0603_1608Metric_Pad1.08x0.95mm_HandSolder, F.Cu at (259.9, 426.2)
- added C432: 0.1uF, Capacitor_SMD:C_0402_1005Metric_Pad0.74x0.62mm_HandSolder, F.Cu at (222.5, 570.4)
- added C433: 0.1uF, Capacitor_SMD:C_0402_1005Metric_Pad0.74x0.62mm_HandSolder, F.Cu at (222.5, 572.4)
- added C434: 0.033uF, Capacitor_SMD:C_0603_1608Metric_Pad1.08x0.95mm_HandSolder, F.Cu at (275.4, 395.6)
- added C435: 0.033uF, Capacitor_SMD:C_0603_1608Metric_Pad1.08x0.95mm_HandSolder, F.Cu at (270.6, 392.6)
- added C436: 1uF, Capacitor_SMD:C_1210_3225Metric_Pad1.33x2.70mm_HandSolder, F.Cu at (256.9, 324.7)
- added C437: 0.01uF, Capacitor_SMD:C_0603_1608Metric_Pad1.08x0.95mm_HandSolder, F.Cu at (157.5, 487.4)
- added C438: 1uF, Capacitor_SMD:C_1210_3225Metric_Pad1.33x2.70mm_HandSolder, F.Cu at (271.7, 324.2)
- added C439: 0.01uF, Capacitor_SMD:C_0603_1608Metric_Pad1.08x0.95mm_HandSolder, F.Cu at (157.5, 490.4)
- added C440: 1uF, Capacitor_SMD:C_1210_3225Metric_Pad1.33x2.70mm_HandSolder, F.Cu at (237.7, 323.7)
- added C441: 1uF, Capacitor_SMD:C_1210_3225Metric_Pad1.33x2.70mm_HandSolder, F.Cu at (231.9, 323.8)
- added C442: 0.01uF, Capacitor_SMD:C_0603_1608Metric_Pad1.08x0.95mm_HandSolder, F.Cu at (153.5, 454.4)
- added C443: 0.01uF, Capacitor_SMD:C_0603_1608Metric_Pad1.08x0.95mm_HandSolder, F.Cu at (158.5, 429.3)
- added C444: 0.033uF, Capacitor_SMD:C_0603_1608Metric_Pad1.08x0.95mm_HandSolder, F.Cu at (250.6, 391.9)
- added C445: 0.033uF, Capacitor_SMD:C_0603_1608Metric_Pad1.08x0.95mm_HandSolder, F.Cu at (248.7, 396.6)
- added C446: 0.1uF, Capacitor_SMD:C_0603_1608Metric_Pad1.08x0.95mm_HandSolder, F.Cu at (251.3, 411.8)
- added C501: 10uF, Capacitor_SMD:C_0603_1608Metric_Pad1.08x0.95mm_HandSolder, F.Cu at (54.6, 276.3)
- added C502: 10uF, Capacitor_SMD:C_0603_1608Metric_Pad1.08x0.95mm_HandSolder, F.Cu at (54.6, 270.3)
- added C503: 10uF, Capacitor_SMD:C_0603_1608Metric_Pad1.08x0.95mm_HandSolder, F.Cu at (229.4, 152.0)
- added C504: 0.1uF, Capacitor_SMD:C_0402_1005Metric_Pad0.74x0.62mm_HandSolder, F.Cu at (243.4, 176.0)
- added C505: 0.1uF, Capacitor_SMD:C_0402_1005Metric_Pad0.74x0.62mm_HandSolder, F.Cu at (112.6, 250.3)
- added C506: 0.1uF, Capacitor_SMD:C_0402_1005Metric_Pad0.74x0.62mm_HandSolder, F.Cu at (232.4, 150.0)
- added C507: 0.1uF, Capacitor_SMD:C_0402_1005Metric_Pad0.74x0.62mm_HandSolder, F.Cu at (232.4, 148.0)
- added C508: 1000pF, Capacitor_SMD:C_0402_1005Metric_Pad0.74x0.62mm_HandSolder, F.Cu at (235.4, 150.0)
- added C509: 2.2uF, Capacitor_SMD:C_0402_1005Metric_Pad0.74x0.62mm_HandSolder, F.Cu at (225.4, 151.0)
- added C510: 1000pF, Capacitor_SMD:C_0402_1005Metric_Pad0.74x0.62mm_HandSolder, F.Cu at (238.4, 153.0)
- added C511: 2.2uF, Capacitor_SMD:C_0402_1005Metric_Pad0.74x0.62mm_HandSolder, F.Cu at (241.4, 161.0)
- added C512: 10uF, Capacitor_SMD:C_1206_3216Metric_Pad1.33x1.80mm_HandSolder, F.Cu at (461.5, 172.1)
- added C513: 10uF, Capacitor_SMD:C_1206_3216Metric_Pad1.33x1.80mm_HandSolder, F.Cu at (244.4, 164.0)
- added C514: 10uF, Capacitor_SMD:C_1206_3216Metric_Pad1.33x1.80mm_HandSolder, F.Cu at (120.6, 182.3)
- added C515: 10uF, Capacitor_SMD:C_1206_3216Metric_Pad1.33x1.80mm_HandSolder, F.Cu at (113.6, 173.3)
- added C516: 100pF, Capacitor_SMD:C_0603_1608Metric_Pad1.08x0.95mm_HandSolder, F.Cu at (445.5, 162.1)
- added C517: 100pF, Capacitor_SMD:C_0603_1608Metric_Pad1.08x0.95mm_HandSolder, F.Cu at (245.4, 156.0)
- added C518: 100pF, Capacitor_SMD:C_0603_1608Metric_Pad1.08x0.95mm_HandSolder, F.Cu at (22.6, 126.3)
- added C519: 100pF, Capacitor_SMD:C_0603_1608Metric_Pad1.08x0.95mm_HandSolder, F.Cu at (27.6, 129.3)
- added C520: 0.1uF, Capacitor_SMD:C_0603_1608Metric_Pad1.08x0.95mm_HandSolder, F.Cu at (450.5, 159.1)
- added C521: 0.1uF, Capacitor_SMD:C_0603_1608Metric_Pad1.08x0.95mm_HandSolder, F.Cu at (451.5, 150.1)
- added C522: 0.1uF, Capacitor_SMD:C_0603_1608Metric_Pad1.08x0.95mm_HandSolder, F.Cu at (139.6, 174.3)
- added C523: 0.1uF, Capacitor_SMD:C_0603_1608Metric_Pad1.08x0.95mm_HandSolder, F.Cu at (44.6, 134.3)
- added C524: 1uF, Capacitor_SMD:C_0603_1608Metric_Pad1.08x0.95mm_HandSolder, F.Cu at (43.6, 128.3)
- added C525: 1uF, Capacitor_SMD:C_0603_1608Metric_Pad1.08x0.95mm_HandSolder, F.Cu at (27.6, 126.3)
- added C526: 0.047uF, Capacitor_SMD:C_0603_1608Metric_Pad1.08x0.95mm_HandSolder, F.Cu at (43.6, 131.3)
- added C527: 1uF, Capacitor_SMD:C_1206_3216Metric_Pad1.33x1.80mm_HandSolder, F.Cu at (133.6, 129.3)
- added C528: 1uF, Capacitor_SMD:C_1206_3216Metric_Pad1.33x1.80mm_HandSolder, F.Cu at (133.6, 174.3)
- added C529: 1000uF, Capacitor_SMD:CP_Elec_16x17.5, F.Cu at (282.2, 96.9)
- added C530: 1uF, Capacitor_SMD:C_1206_3216Metric_Pad1.33x1.80mm_HandSolder, F.Cu at (133.6, 132.3)
- added C531: 1uF, Capacitor_SMD:C_1206_3216Metric_Pad1.33x1.80mm_HandSolder, F.Cu at (133.6, 150.3)
- added C532: 1000uF, Capacitor_SMD:CP_Elec_16x17.5, F.Cu at (280.3, 75.5)
- added C533: 0.033uF, Capacitor_SMD:C_0603_1608Metric_Pad1.08x0.95mm_HandSolder, F.Cu at (43.6, 152.3)
- added C534: 0.033uF, Capacitor_SMD:C_0603_1608Metric_Pad1.08x0.95mm_HandSolder, F.Cu at (40.6, 146.3)
- added C535: 0.033uF, Capacitor_SMD:C_0603_1608Metric_Pad1.08x0.95mm_HandSolder, F.Cu at (38.6, 149.3)
- added C536: 0.033uF, Capacitor_SMD:C_0603_1608Metric_Pad1.08x0.95mm_HandSolder, F.Cu at (45.6, 146.3)
- added C537: 1uF, Capacitor_SMD:C_1210_3225Metric_Pad1.33x2.70mm_HandSolder, F.Cu at (450.5, 166.1)
- added C538: 0.01uF, Capacitor_SMD:C_0603_1608Metric_Pad1.08x0.95mm_HandSolder, F.Cu at (19.6, 213.3)
- added C539: 1uF, Capacitor_SMD:C_1210_3225Metric_Pad1.33x2.70mm_HandSolder, F.Cu at (456.5, 161.1)
- added C540: 0.01uF, Capacitor_SMD:C_0603_1608Metric_Pad1.08x0.95mm_HandSolder, F.Cu at (460.5, 178.1)
- added C541: 1uF, Capacitor_SMD:C_1210_3225Metric_Pad1.33x2.70mm_HandSolder, F.Cu at (240.4, 168.0)
- added C542: 0.01uF, Capacitor_SMD:C_0603_1608Metric_Pad1.08x0.95mm_HandSolder, F.Cu at (-14.4, 168.3)
- added C543: 1uF, Capacitor_SMD:C_1210_3225Metric_Pad1.33x2.70mm_HandSolder, F.Cu at (244.4, 173.0)
- added C544: 0.01uF, Capacitor_SMD:C_0603_1608Metric_Pad1.08x0.95mm_HandSolder, F.Cu at (27.6, 135.3)
- added C601: 10uF, Capacitor_SMD:C_0603_1608Metric_Pad1.08x0.95mm_HandSolder, F.Cu at (127.6, 275.3)
- added C601: 10uF, Capacitor_SMD:C_0603_1608Metric_Pad1.08x0.95mm_HandSolder, F.Cu at (210.8, 115.8)
- added C602: 10uF, Capacitor_SMD:C_0603_1608Metric_Pad1.08x0.95mm_HandSolder, F.Cu at (54.6, 264.3)
- added C603: 0.1uF, Capacitor_SMD:C_0402_1005Metric_Pad0.74x0.62mm_HandSolder, F.Cu at (127.6, 279.3)
- added C604: 0.1uF, Capacitor_SMD:C_0402_1005Metric_Pad0.74x0.62mm_HandSolder, F.Cu at (110.6, 246.3)
- added C605: 10uF, Capacitor_SMD:C_0603_1608Metric_Pad1.08x0.95mm_HandSolder, F.Cu at (54.6, 267.3)
- added C606: 0.1uF, Capacitor_SMD:C_0402_1005Metric_Pad0.74x0.62mm_HandSolder, F.Cu at (54.6, 285.3)
- added C607: 2.2uF, Capacitor_SMD:C_0402_1005Metric_Pad0.74x0.62mm_HandSolder, F.Cu at (114.6, 259.3)
- added C608: 0.1uF, Capacitor_SMD:C_0402_1005Metric_Pad0.74x0.62mm_HandSolder, F.Cu at (138.6, 241.3)
- added C609: 2.2uF, Capacitor_SMD:C_0402_1005Metric_Pad0.74x0.62mm_HandSolder, F.Cu at (117.6, 259.3)
- added C610: 1000pF, Capacitor_SMD:C_0402_1005Metric_Pad0.74x0.62mm_HandSolder, F.Cu at (118.6, 279.3)
- added C611: 1000pF, Capacitor_SMD:C_0402_1005Metric_Pad0.74x0.62mm_HandSolder, F.Cu at (113.6, 277.3)
- added C612: 10uF, Capacitor_SMD:C_1206_3216Metric_Pad1.33x1.80mm_HandSolder, F.Cu at (229.4, 223.0)
- added C613: 10uF, Capacitor_SMD:C_1206_3216Metric_Pad1.33x1.80mm_HandSolder, F.Cu at (143.6, 240.3)
- added C614: 10uF, Capacitor_SMD:C_1206_3216Metric_Pad1.33x1.80mm_HandSolder, F.Cu at (122.6, 228.3)
- added C615: 10uF, Capacitor_SMD:C_1206_3216Metric_Pad1.33x1.80mm_HandSolder, F.Cu at (143.6, 220.3)
- added C616: 100pF, Capacitor_SMD:C_0603_1608Metric_Pad1.08x0.95mm_HandSolder, F.Cu at (150.7, 277.5)
- added C617: 100pF, Capacitor_SMD:C_0603_1608Metric_Pad1.08x0.95mm_HandSolder, F.Cu at (147.6, 274.3)
- added C618: 100pF, Capacitor_SMD:C_0603_1608Metric_Pad1.08x0.95mm_HandSolder, F.Cu at (132.6, 274.3)
- added C619: 100pF, Capacitor_SMD:C_0603_1608Metric_Pad1.08x0.95mm_HandSolder, F.Cu at (227.4, 158.0)
- added C620: 0.1uF, Capacitor_SMD:C_0603_1608Metric_Pad1.08x0.95mm_HandSolder, F.Cu at (146.6, 166.3)
- added C621: 0.1uF, Capacitor_SMD:C_0603_1608Metric_Pad1.08x0.95mm_HandSolder, F.Cu at (139.6, 168.3)
- added C622: 0.1uF, Capacitor_SMD:C_0603_1608Metric_Pad1.08x0.95mm_HandSolder, F.Cu at (139.6, 159.3)
- added C623: 0.047uF, Capacitor_SMD:C_0603_1608Metric_Pad1.08x0.95mm_HandSolder, F.Cu at (228.4, 234.0)
- added C624: 1uF, Capacitor_SMD:C_0603_1608Metric_Pad1.08x0.95mm_HandSolder, F.Cu at (234.4, 230.0)
- added C625: 1uF, Capacitor_SMD:C_0603_1608Metric_Pad1.08x0.95mm_HandSolder, F.Cu at (221.4, 150.0)
- added C626: 1uF, Capacitor_SMD:C_1206_3216Metric_Pad1.33x1.80mm_HandSolder, F.Cu at (133.6, 135.3)
- added C627: 1uF, Capacitor_SMD:C_1206_3216Metric_Pad1.33x1.80mm_HandSolder, F.Cu at (133.6, 168.3)
- added C628: 1uF, Capacitor_SMD:C_1206_3216Metric_Pad1.33x1.80mm_HandSolder, F.Cu at (133.6, 156.3)
- added C629: 1uF, Capacitor_SMD:C_1206_3216Metric_Pad1.33x1.80mm_HandSolder, F.Cu at (133.6, 162.3)
- added C630: 1000uF, Capacitor_SMD:CP_Elec_16x17.5, F.Cu at (325.3, 103.1)
- added C631: 1000uF, Capacitor_SMD:CP_Elec_16x17.5, F.Cu at (325.0, 74.0)
- added C632: 0.033uF, Capacitor_SMD:C_0603_1608Metric_Pad1.08x0.95mm_HandSolder, F.Cu at (237.4, 246.0)
- added C633: 0.033uF, Capacitor_SMD:C_0603_1608Metric_Pad1.08x0.95mm_HandSolder, F.Cu at (232.4, 161.0)
- added C634: 0.033uF, Capacitor_SMD:C_0603_1608Metric_Pad1.08x0.95mm_HandSolder, F.Cu at (459.5, 219.1)
- added C635: 0.033uF, Capacitor_SMD:C_0603_1608Metric_Pad1.08x0.95mm_HandSolder, F.Cu at (227.4, 161.0)
- added C636: 0.1uF, Capacitor_SMD:C_0603_1608Metric_Pad1.08x0.95mm_HandSolder, F.Cu at (222.4, 147.0)
- added C637: 1uF, Capacitor_SMD:C_1210_3225Metric_Pad1.33x2.70mm_HandSolder, F.Cu at (114.6, 240.3)
- added C638: 1uF, Capacitor_SMD:C_1210_3225Metric_Pad1.33x2.70mm_HandSolder, F.Cu at (149.6, 258.3)
- added C639: 1uF, Capacitor_SMD:C_1210_3225Metric_Pad1.33x2.70mm_HandSolder, F.Cu at (133.6, 259.3)
- added C640: 1uF, Capacitor_SMD:C_1210_3225Metric_Pad1.33x2.70mm_HandSolder, F.Cu at (127.6, 241.3)
- added C641: 0.01uF, Capacitor_SMD:C_0603_1608Metric_Pad1.08x0.95mm_HandSolder, F.Cu at (150.6, 262.3)
- added C642: 0.01uF, Capacitor_SMD:C_0603_1608Metric_Pad1.08x0.95mm_HandSolder, F.Cu at (150.6, 265.3)
- added C643: 0.01uF, Capacitor_SMD:C_0603_1608Metric_Pad1.08x0.95mm_HandSolder, F.Cu at (142.6, 274.3)
- added C644: 0.01uF, Capacitor_SMD:C_0603_1608Metric_Pad1.08x0.95mm_HandSolder, F.Cu at (144.6, 160.3)
- added C701: 10uF, Capacitor_SMD:C_0603_1608Metric_Pad1.08x0.95mm_HandSolder, F.Cu at (127.6, 178.3)
- added C702: 10uF, Capacitor_SMD:C_0603_1608Metric_Pad1.08x0.95mm_HandSolder, F.Cu at (117.6, 161.3)
- added C703: 0.1uF, Capacitor_SMD:C_0402_1005Metric_Pad0.74x0.62mm_HandSolder, F.Cu at (127.6, 164.3)
- added C704: 0.1uF, Capacitor_SMD:C_0402_1005Metric_Pad0.74x0.62mm_HandSolder, F.Cu at (117.6, 151.3)
- added C705: 10uF, Capacitor_SMD:C_0603_1608Metric_Pad1.08x0.95mm_HandSolder, F.Cu at (117.6, 155.3)
- added C706: 0.1uF, Capacitor_SMD:C_0402_1005Metric_Pad0.74x0.62mm_HandSolder, F.Cu at (117.6, 153.3)
- added C707: 2.2uF, Capacitor_SMD:C_0402_1005Metric_Pad0.74x0.62mm_HandSolder, F.Cu at (125.6, 156.3)
- added C708: 0.1uF, Capacitor_SMD:C_0402_1005Metric_Pad0.74x0.62mm_HandSolder, F.Cu at (128.6, 156.3)
- added C709: 2.2uF, Capacitor_SMD:C_0402_1005Metric_Pad0.74x0.62mm_HandSolder, F.Cu at (131.6, 212.3)
- added C710: 1000pF, Capacitor_SMD:C_0402_1005Metric_Pad0.74x0.62mm_HandSolder, F.Cu at (241.4, 152.0)
- added C711: 1000pF, Capacitor_SMD:C_0402_1005Metric_Pad0.74x0.62mm_HandSolder, F.Cu at (15.6, 220.3)
- added C712: 10uF, Capacitor_SMD:C_1206_3216Metric_Pad1.33x1.80mm_HandSolder, F.Cu at (126.6, 172.3)
- added C713: 10uF, Capacitor_SMD:C_1206_3216Metric_Pad1.33x1.80mm_HandSolder, F.Cu at (65.6, 159.3)
- added C714: 10uF, Capacitor_SMD:C_1206_3216Metric_Pad1.33x1.80mm_HandSolder, F.Cu at (13.6, 212.3)
- added C715: 10uF, Capacitor_SMD:C_1206_3216Metric_Pad1.33x1.80mm_HandSolder, F.Cu at (23.6, 222.3)
- added C716: 100pF, Capacitor_SMD:C_0603_1608Metric_Pad1.08x0.95mm_HandSolder, F.Cu at (8.57, 159.3)
- added C717: 100pF, Capacitor_SMD:C_0603_1608Metric_Pad1.08x0.95mm_HandSolder, F.Cu at (74.6, 156.3)
- added C718: 100pF, Capacitor_SMD:C_0603_1608Metric_Pad1.08x0.95mm_HandSolder, F.Cu at (7.57, 221.3)
- added C719: 100pF, Capacitor_SMD:C_0603_1608Metric_Pad1.08x0.95mm_HandSolder, F.Cu at (12.6, 223.3)
- added C720: 0.1uF, Capacitor_SMD:C_0603_1608Metric_Pad1.08x0.95mm_HandSolder, F.Cu at (-5.43, 200.3)
- added C721: 0.1uF, Capacitor_SMD:C_0603_1608Metric_Pad1.08x0.95mm_HandSolder, F.Cu at (450.5, 156.1)
- added C722: 0.1uF, Capacitor_SMD:C_0603_1608Metric_Pad1.08x0.95mm_HandSolder, F.Cu at (139.6, 177.3)
- added C723: 0.047uF, Capacitor_SMD:C_0603_1608Metric_Pad1.08x0.95mm_HandSolder, F.Cu at (1.57, 151.3)
- added C724: 1uF, Capacitor_SMD:C_0603_1608Metric_Pad1.08x0.95mm_HandSolder, F.Cu at (7.57, 218.3)
- added C725: 1uF, Capacitor_SMD:C_0603_1608Metric_Pad1.08x0.95mm_HandSolder, F.Cu at (-3.43, 152.3)
- added C726: 1uF, Capacitor_SMD:C_1206_3216Metric_Pad1.33x1.80mm_HandSolder, F.Cu at (133.6, 171.3)
- added C727: 1uF, Capacitor_SMD:C_1206_3216Metric_Pad1.33x1.80mm_HandSolder, F.Cu at (133.6, 165.3)
- added C728: 1uF, Capacitor_SMD:C_1206_3216Metric_Pad1.33x1.80mm_HandSolder, F.Cu at (133.6, 159.3)
- added C729: 1uF, Capacitor_SMD:C_1206_3216Metric_Pad1.33x1.80mm_HandSolder, F.Cu at (133.6, 147.3)
- added C730: 1000uF, Capacitor_SMD:CP_Elec_16x17.5, F.Cu at (372.3, 102.1)
- added C731: 1000uF, Capacitor_SMD:CP_Elec_16x17.5, F.Cu at (369.5, 80.5)
- added C732: 0.033uF, Capacitor_SMD:C_0603_1608Metric_Pad1.08x0.95mm_HandSolder, F.Cu at (-16.4, 187.3)
- added C733: 0.033uF, Capacitor_SMD:C_0603_1608Metric_Pad1.08x0.95mm_HandSolder, F.Cu at (64.6, 162.3)
- added C734: 0.033uF, Capacitor_SMD:C_0603_1608Metric_Pad1.08x0.95mm_HandSolder, F.Cu at (8.57, 206.3)
- added C735: 0.033uF, Capacitor_SMD:C_0603_1608Metric_Pad1.08x0.95mm_HandSolder, F.Cu at (-9.43, 166.3)
- added C736: 0.1uF, Capacitor_SMD:C_0603_1608Metric_Pad1.08x0.95mm_HandSolder, F.Cu at (-14.4, 174.3)
- added C737: 1uF, Capacitor_SMD:C_1210_3225Metric_Pad1.33x2.70mm_HandSolder, F.Cu at (76.6, 168.3)
- added C738: 1uF, Capacitor_SMD:C_1210_3225Metric_Pad1.33x2.70mm_HandSolder, F.Cu at (-6.43, 194.3)
- added C739: 1uF, Capacitor_SMD:C_1210_3225Metric_Pad1.33x2.70mm_HandSolder, F.Cu at (83.6, 176.3)
- added C740: 1uF, Capacitor_SMD:C_1210_3225Metric_Pad1.33x2.70mm_HandSolder, F.Cu at (70.6, 190.3)
- added C741: 0.01uF, Capacitor_SMD:C_0603_1608Metric_Pad1.08x0.95mm_HandSolder, F.Cu at (8.57, 209.3)
- added C742: 0.01uF, Capacitor_SMD:C_0603_1608Metric_Pad1.08x0.95mm_HandSolder, F.Cu at (-16.4, 190.3)
- added C743: 0.01uF, Capacitor_SMD:C_0603_1608Metric_Pad1.08x0.95mm_HandSolder, F.Cu at (17.6, 225.3)
- added C744: 0.01uF, Capacitor_SMD:C_0603_1608Metric_Pad1.08x0.95mm_HandSolder, F.Cu at (34.6, 135.3)
- added C801: 10uF, Capacitor_SMD:C_0603_1608Metric_Pad1.08x0.95mm_HandSolder, F.Cu at (117.6, 179.3)
- added C802: 10uF, Capacitor_SMD:C_0603_1608Metric_Pad1.08x0.95mm_HandSolder, F.Cu at (117.6, 158.3)
- added C803: 0.1uF, Capacitor_SMD:C_0402_1005Metric_Pad0.74x0.62mm_HandSolder, F.Cu at (123.6, 203.3)
- added C804: 0.1uF, Capacitor_SMD:C_0402_1005Metric_Pad0.74x0.62mm_HandSolder, F.Cu at (142.6, 209.3)
- added C805: 10uF, Capacitor_SMD:C_0603_1608Metric_Pad1.08x0.95mm_HandSolder, F.Cu at (137.6, 210.3)
- added C806: 0.1uF, Capacitor_SMD:C_0402_1005Metric_Pad0.74x0.62mm_HandSolder, F.Cu at (126.6, 207.3)
- added C807: 2.2uF, Capacitor_SMD:C_0402_1005Metric_Pad0.74x0.62mm_HandSolder, F.Cu at (127.6, 162.3)
- added C808: 0.1uF, Capacitor_SMD:C_0402_1005Metric_Pad0.74x0.62mm_HandSolder, F.Cu at (128.6, 180.3)
- added C809: 2.2uF, Capacitor_SMD:C_0402_1005Metric_Pad0.74x0.62mm_HandSolder, F.Cu at (123.6, 174.3)
- added C810: 1000pF, Capacitor_SMD:C_0402_1005Metric_Pad0.74x0.62mm_HandSolder, F.Cu at (122.6, 165.3)
- added C811: 1000pF, Capacitor_SMD:C_0402_1005Metric_Pad0.74x0.62mm_HandSolder, F.Cu at (121.6, 158.3)
- added C812: 10uF, Capacitor_SMD:C_1206_3216Metric_Pad1.33x1.80mm_HandSolder, F.Cu at (117.6, 185.3)
- added C813: 10uF, Capacitor_SMD:C_1206_3216Metric_Pad1.33x1.80mm_HandSolder, F.Cu at (131.6, 197.3)
- added C814: 10uF, Capacitor_SMD:C_1206_3216Metric_Pad1.33x1.80mm_HandSolder, F.Cu at (113.6, 176.3)
- added C815: 10uF, Capacitor_SMD:C_1206_3216Metric_Pad1.33x1.80mm_HandSolder, F.Cu at (120.6, 176.3)
- added C816: 100pF, Capacitor_SMD:C_0603_1608Metric_Pad1.08x0.95mm_HandSolder, F.Cu at (108.6, 164.3)
- added C817: 100pF, Capacitor_SMD:C_0603_1608Metric_Pad1.08x0.95mm_HandSolder, F.Cu at (126.6, 166.3)
- added C818: 100pF, Capacitor_SMD:C_0603_1608Metric_Pad1.08x0.95mm_HandSolder, F.Cu at (113.6, 167.3)
- added C819: 100pF, Capacitor_SMD:C_0603_1608Metric_Pad1.08x0.95mm_HandSolder, F.Cu at (127.6, 169.3)
- added C820: 0.1uF, Capacitor_SMD:C_0603_1608Metric_Pad1.08x0.95mm_HandSolder, F.Cu at (145.6, 172.3)
- added C821: 0.1uF, Capacitor_SMD:C_0603_1608Metric_Pad1.08x0.95mm_HandSolder, F.Cu at (139.6, 165.3)
- added C822: 0.1uF, Capacitor_SMD:C_0603_1608Metric_Pad1.08x0.95mm_HandSolder, F.Cu at (139.6, 162.3)
- added C823: 0.047uF, Capacitor_SMD:C_0603_1608Metric_Pad1.08x0.95mm_HandSolder, F.Cu at (-8.43, 160.3)
- added C824: 1uF, Capacitor_SMD:C_0603_1608Metric_Pad1.08x0.95mm_HandSolder, F.Cu at (22.6, 132.3)
- added C825: 1uF, Capacitor_SMD:C_0603_1608Metric_Pad1.08x0.95mm_HandSolder, F.Cu at (22.6, 129.3)
- added C826: 1uF, Capacitor_SMD:C_1206_3216Metric_Pad1.33x1.80mm_HandSolder, F.Cu at (133.6, 138.3)
- added C827: 1uF, Capacitor_SMD:C_1206_3216Metric_Pad1.33x1.80mm_HandSolder, F.Cu at (133.6, 141.3)
- added C828: 1uF, Capacitor_SMD:C_1206_3216Metric_Pad1.33x1.80mm_HandSolder, F.Cu at (133.6, 144.3)
- added C829: 1uF, Capacitor_SMD:C_1206_3216Metric_Pad1.33x1.80mm_HandSolder, F.Cu at (133.6, 126.3)
- added C830: 1000uF, Capacitor_SMD:CP_Elec_16x17.5, F.Cu at (421.1, 106.8)
- added C831: 1000uF, Capacitor_SMD:CP_Elec_16x17.5, F.Cu at (420.8, 83.8)
- added C832: 0.033uF, Capacitor_SMD:C_0603_1608Metric_Pad1.08x0.95mm_HandSolder, F.Cu at (22.6, 135.3)
- added C833: 0.033uF, Capacitor_SMD:C_0603_1608Metric_Pad1.08x0.95mm_HandSolder, F.Cu at (-4.43, 166.3)
- added C834: 0.033uF, Capacitor_SMD:C_0603_1608Metric_Pad1.08x0.95mm_HandSolder, F.Cu at (38.6, 142.3)
- added C835: 0.033uF, Capacitor_SMD:C_0603_1608Metric_Pad1.08x0.95mm_HandSolder, F.Cu at (38.6, 152.3)
- added C836: 0.1uF, Capacitor_SMD:C_0603_1608Metric_Pad1.08x0.95mm_HandSolder, F.Cu at (-4.43, 163.3)
- added C837: 1uF, Capacitor_SMD:C_1210_3225Metric_Pad1.33x2.70mm_HandSolder, F.Cu at (223.4, 154.0)
- added C838: 1uF, Capacitor_SMD:C_1210_3225Metric_Pad1.33x2.70mm_HandSolder, F.Cu at (221.4, 159.0)
- added C839: 1uF, Capacitor_SMD:C_1210_3225Metric_Pad1.33x2.70mm_HandSolder, F.Cu at (2.57, 158.3)
- added C840: 1uF, Capacitor_SMD:C_1210_3225Metric_Pad1.33x2.70mm_HandSolder, F.Cu at (-13.4, 194.3)
- added C841: 0.01uF, Capacitor_SMD:C_0603_1608Metric_Pad1.08x0.95mm_HandSolder, F.Cu at (151.6, 166.3)
- added C842: 0.01uF, Capacitor_SMD:C_0603_1608Metric_Pad1.08x0.95mm_HandSolder, F.Cu at (10.6, 144.3)
- added C843: 0.01uF, Capacitor_SMD:C_0603_1608Metric_Pad1.08x0.95mm_HandSolder, F.Cu at (8.57, 137.3)
- added C844: 0.01uF, Capacitor_SMD:C_0603_1608Metric_Pad1.08x0.95mm_HandSolder, F.Cu at (-9.43, 154.3)
- added C901: 10uF, Capacitor_SMD:C_0603_1608Metric_Pad1.08x0.95mm_HandSolder, F.Cu at (462.5, 189.1)
- added C902: 10uF, Capacitor_SMD:C_0603_1608Metric_Pad1.08x0.95mm_HandSolder, F.Cu at (183.9, 132.2)
- added C903: 0.1uF, Capacitor_SMD:C_0402_1005Metric_Pad0.74x0.62mm_HandSolder, F.Cu at (443.5, 202.1)
- added C904: 0.1uF, Capacitor_SMD:C_0402_1005Metric_Pad0.74x0.62mm_HandSolder, F.Cu at (184.9, 127.2)
- added C905: 10uF, Capacitor_SMD:C_0603_1608Metric_Pad1.08x0.95mm_HandSolder, F.Cu at (462.5, 186.1)
- added C906: 0.1uF, Capacitor_SMD:C_0402_1005Metric_Pad0.74x0.62mm_HandSolder, F.Cu at (247.4, 241.0)
- added C907: 2.2uF, Capacitor_SMD:C_0402_1005Metric_Pad0.74x0.62mm_HandSolder, F.Cu at (465.5, 213.1)
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Other:
- board outline added: 800 x 85 mm

Commit message: Modification d'empreinte et routage de sortie audio
Parts:
- C422, C425: footprint Capacitor_SMD:CP_Elec_16x17.5 -> NewLibrary:CAP_EEVFK1H102M
- C432, C433, C437, C439, C442, C443, R210, R322, R327, R419, R420, R421, R422, U403, U404: moved to B.Cu
- J401: value Surrond Left+ -> SL+
- J402: value Surrond Left- -> SL-
- J403: value Surrond Right+ -> SR+
- J404: value SurroundRight- -> SR-
- moved R327 344.2 mm to (230.2, 476.7)
- moved R322 338.7 mm to (227.0, 475.8), turned to 180 degrees
- moved R210 303.9 mm to (235.4, 477.8)
- moved R301 293.5 mm to (272.1, 484.2), turned to -90 degrees
- moved R313 265.9 mm to (268.5, 484.2), turned to -90 degrees
- moved R307 265.8 mm to (264.9, 484.2), turned to -90 degrees
- moved C405 210.0 mm to (262.9, 463.0), turned to -90 degrees
- moved C437 205.1 mm to (265.2, 313.0), turned to 90 degrees
- moved C439 200.3 mm to (251.1, 313.4), turned to -90 degrees
- moved R404 198.2 mm to (262.5, 472.6)
- moved R421 191.8 mm to (248.7, 303.0), turned to 90 degrees
- moved R408 187.6 mm to (259.2, 462.2)
- moved C404 184.5 mm to (286.7, 481.8)
- moved R407 183.4 mm to (262.6, 468.9)
- moved C442 183.0 mm to (248.6, 298.1), turned to 90 degrees
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Routing:
- net Net-(R307-Pad1): track 0.00 -> 137.0 mm
- net GND: track 0.00 -> 12.0 mm
- net Net-(U402-BST_C): track 0.00 -> 3.95 mm
- net Net-(JP402-C): track 0.00 -> 0.86 mm
- net 3.3V-4: track 0.00 -> 0.65 mm
- net /Surrond_Channel/DAC1L+: track 0.00 -> 0.59 mm
- added copper zone on F.Cu, net /Surrond_Channel/Surrond Right+
- added copper zone on F.Cu, net /Surrond_Channel/SurroundRight-
Other:
- board text added: "SR+"
- board text added: "SR-"

Commit message: Continuation du routage
Parts:
- moved U402 40.5 mm to (248.8, 364.1)
- moved C434 39.8 mm to (258.1, 360.2), turned to 180 degrees
- moved C445 38.0 mm to (239.4, 360.2), turned to 0 degrees
- moved C435 36.8 mm to (258.1, 357.9), turned to 180 degrees
- moved C444 35.8 mm to (239.4, 357.9)
- moved C427 35.7 mm to (235.2, 374.9)
- moved C428 35.7 mm to (259.2, 379.3)
- moved L401 35.7 mm to (259.3, 383.6)
- moved C446 35.7 mm to (238.5, 378.5)
- moved C426 35.7 mm to (259.9, 375.2)
- moved C424 32.1 mm to (257.2, 354.4), turned to 180 degrees
- moved C423 31.6 mm to (251.8, 354.4)
- moved C421 31.5 mm to (245.8, 354.4), turned to 180 degrees
- moved C420 31.2 mm to (240.3, 354.4)
- moved R420 25.9 mm to (255.2, 292.1)
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Connections:
- L402 pad 1: /Surrond_Channel/OUT1A -> /Surrond_Channel/OUT1B
- L402 pad 2: /Surrond_Channel/Surrond Left+ -> /Surrond_Channel/Surrond Left-
- L402 pad 3: /Surrond_Channel/Surrond Left- -> /Surrond_Channel/Surrond Left+
- L402 pad 4: /Surrond_Channel/OUT1B -> /Surrond_Channel/OUT1A
- L403 pad 1: /Surrond_Channel/OUT1C -> /Surrond_Channel/OUT1D
- L403 pad 2: /Surrond_Channel/Surrond Right+ -> /Surrond_Channel/SurroundRight-
- L403 pad 3: /Surrond_Channel/SurroundRight- -> /Surrond_Channel/Surrond Right+
- L403 pad 4: /Surrond_Channel/OUT1D -> /Surrond_Channel/OUT1C
Routing:
- net PVDD: track 0.00 -> 6.69 mm
- net Net-(U402-BST_B): track 0.00 -> 4.22 mm
- net /Surrond_Channel/OUT1D: track 0.00 -> 3.35 mm
- net /Surrond_Channel/OUT1B: track 0.00 -> 3.11 mm
- net /Surrond_Channel/OUT1C: track 0.00 -> 3.10 mm
- net /Surrond_Channel/OUT1A: track 0.00 -> 2.53 mm
- net Net-(U402-BST_A): track 0.00 -> 1.87 mm
- net Net-(U402-BST_D): track 0.00 -> 1.87 mm
- added copper zone on F.Cu, net /Surrond_Channel/OUT1A
- added copper zone on F.Cu, net /Surrond_Channel/OUT1D
- added copper zone on F.Cu, net /Surrond_Channel/Surrond Left+
- added copper zone on F.Cu, net /Surrond_Channel/Surrond Left-
- added copper zone on F.Cu, net PVDD
Other:
- copper layers 2 -> 4

Commit message: suite du routage
Parts:
- U402: footprint NewLibrary:DDV0044D_N -> Package_SO:HTSSOP-44-1EP_6.1x14mm_P0.635mm_EP5.2x14mm_Mask4.31x8.26mm_ThermalVias
- moved JP401 70.9 mm to (269.4, 378.2)
- moved JP402 68.6 mm to (259.1, 378.2)
- moved JP403 67.9 mm to (237.2, 378.2)
- moved JP404 67.8 mm to (226.9, 378.2)
- moved C413 66.3 mm to (262.7, 373.6)
- moved R413 64.0 mm to (262.7, 371.9)
- moved C415 63.7 mm to (253.2, 375.0)
- moved C412 63.2 mm to (267.9, 373.2), turned to 180 degrees
- moved C414 62.7 mm to (257.6, 373.2), turned to 180 degrees
- moved R414 62.6 mm to (253.2, 373.2)
- moved C419 62.5 mm to (233.6, 373.4), turned to 180 degrees
- moved R416 61.1 mm to (233.6, 371.6), turned to 180 degrees
- moved C418 59.0 mm to (228.5, 373.2)
- moved C417 58.8 mm to (243.4, 375.0), turned to 180 degrees
- moved R417 58.2 mm to (247.0, 377.7), turned to 180 degrees
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Routing:
- net /Surrond_Channel/OUT1B: track 3.11 -> 40.5 mm, vias 0 -> 12
- net /Surrond_Channel/OUT1C: track 3.10 -> 35.7 mm, vias 0 -> 8
- net /Surrond_Channel/OUT1D: track 3.35 -> 35.8 mm, vias 0 -> 12
- net /Surrond_Channel/OUT1A: track 2.53 -> 33.8 mm, vias 0 -> 8
- net /Surrond_Channel/INPUTD1: track 0.20 -> 15.3 mm
- net /Surrond_Channel/INPUTA1: track 0.07 -> 12.8 mm
- net Net-(U402-OC_ADJ): track 0.00 -> 11.5 mm
- net 12V: track 0.00 -> 10.8 mm, vias 0 -> 1
- net Net-(U402-FREQ_ADJ): track 0.00 -> 9.56 mm
- net /Surrond_Channel/VDD1: track 0.00 -> 8.48 mm
- net /Surrond_Channel/INPUTC1: track 0.13 -> 8.19 mm
- net /Surrond_Channel/INPUTB1: track 0.07 -> 7.20 mm
- net PVDD: track 6.69 -> 0.00 mm
- net Net-(U402-C_START): track 0.00 -> 6.53 mm
- net Net-(U402-AVDD): track 0.00 -> 4.51 mm
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- added copper zone on F.Cu, net /Surrond_Channel/OUT1B
- added copper zone on F.Cu, net /Surrond_Channel/OUT1C
