File: Amplificateur_Audio/Amplificateur_Audio_Custom/Amplificateur_Audio.kicad_pcb (KiCad board)
At the start: 4 copper layers, 800 x 85 mm, 859 parts, among them J1101 SURROUND-LEFT, J1102 UPMIX-LEFT, J1103 FR-TWEETER, J1104 FL-TWEETER, J1105 CENTER-TWEETER, J1106 SURROUND-RIGHT, J1107 UPMIX-RIGHT, J1108 FR-WOOFER, J1109 FL-WOOFER, J1110 CENTER-WOOFER, J1111 Analog OUTPUT Connector, J201 JTAG, J202 Conn_01x02, J203 Conn_02x08_Odd_Even, J301 Conn_02x10_Odd_Even, J401 SL+, J402 SL-, J403 SR+, J404 SR-, J405 Analog input Connector, J501 UP LEFT+, J502 UP LEFT-, J503 UP RIGHT+, J504 UP RIGHT-, J601 Front Right Tweeter+, J602 Front Right Tweeter-, J603 Front Right Woofer+, J604 Front Right Woofer-, J701 Front Left Tweeter+, J702 Front Left Tweeter-, J703 Front Left Woofer+, J704 Front Left Woofer-, J801 Center Tweeter+, J802 Center Tweeter-, J803 Center Woofer+, J804 Center Woofer-, J901 I2S-OUT, J902 SUBOUT, Q201 NPN, Q202 NPN, Q203 NPN, Q204 NPN, Q205 NPN, Q206 NPN, Q301 NMOS, Q302 NMOS, SW201 MUTE, SW202 VOL+, SW203 VOL-, SW204 MODE1, SW205 MODE2, SW206 MODE3, SW207 MODE4, SW208 LOAD, SW209 RESET, U1101 NE5532AD, U1102 NE5532AD, U1103 NE5532AD, U1104 NE5532AD, U1105 NE5532AD, U1106 NE5532AD, U1107 NE5532AD, U1108 NE5532AD, U1109 NE5532AD, U1110 NE5532AD, U201 MSP430F5234IRGZ, U202 TCA6408ARSVR, U203 24LC512, U204 TCA9548ARGER, U301 74LVC1G125, U302 74LVC1G125, U303 74LVC1G125, U304 74LVC1G125, U305 74LVC1G125, U306 74LVC1G125, U307 74LVC1G125, U308 74LVC1G125, U309 74LVC1G125, U310 74LVC1G125, U401 PCM5252RHBR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

Commit message: Suite routage
Parts:
- moved U401 46.2 mm to (249.1, 388.4), turned to 180 degrees
- moved R412 38.1 mm to (240.7, 382.7)
- moved C411 35.0 mm to (238.4, 383.5)
- moved C401 35.0 mm to (261.5, 398.1)
- moved C403 35.0 mm to (261.3, 408.4)
- moved C406 35.0 mm to (238.8, 391.6)
- moved C409 35.0 mm to (258.8, 414.2)
- moved R301 35.0 mm to (243.8, 413.7)
- moved R401 35.0 mm to (234.0, 405.7)
- moved R402 35.0 mm to (233.9, 409.4)
- moved R403 35.0 mm to (254.3, 413.6)
- moved R406 35.0 mm to (250.8, 413.7)
- moved C405 35.0 mm to (234.6, 392.5)
- moved R307 35.0 mm to (236.5, 413.6)
- moved R408 35.0 mm to (230.9, 391.7)
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Routing:
- net /Surrond_Channel/DAC1R-: track 0.27 -> 14.5 mm
- net /Surrond_Channel/DAC1R+: track 0.00 -> 4.35 mm
- net /Surrond_Channel/DAC1L+: track 0.59 -> 0.00 mm
Other:
- board text added: "embrasse moi bordel"
- board text added: "je rigole je t m"
- board text added: "mon amour je t'aime énormément t'es trop sexy quand tu me parles de ton taf même si je capte R je t'aime"

Commit message: Suite routage
Parts:
- moved C404 27.1 mm to (247.4, 386.5)
- moved R408 13.0 mm to (242.5, 386.0), turned to 180 degrees
- moved C405 11.8 mm to (244.9, 386.8), turned to 90 degrees
- moved C406 6.96 mm to (232.2, 389.4), turned to 90 degrees
- moved C410 3.58 mm to (259.8, 383.5)
- moved R410 3.51 mm to (257.5, 382.7)
- moved R409 3.49 mm to (257.5, 384.4)
- moved U401 2.35 mm to (248.7, 390.7)
- moved R411 1.74 mm to (240.7, 382.7)
- moved R412 1.72 mm to (240.7, 384.4)
- turned C411 to -90 degrees
Routing:
- net /Surrond_Channel/DAC1L+: track 0.00 -> 15.4 mm
- net /Surrond_Channel/OUTRN1: track 0.00 -> 11.0 mm
- net GND: track 11.5 -> 0.78 mm
- net /Surrond_Channel/OUTRP1: track 0.00 -> 10.1 mm
- net /Surrond_Channel/OUTLN1: track 0.00 -> 9.78 mm
- net /Surrond_Channel/OUTLP1: track 0.00 -> 8.42 mm
- net Net-(U401-AVDD): track 0.00 -> 6.64 mm
- net /Surrond_Channel/DAC1L-: track 0.00 -> 5.88 mm
- net /Surrond_Channel/DAC1R+: track 4.35 -> 9.54 mm, vias 0 -> 2
- net /Surrond_Channel/DAC1R-: track 14.5 -> 11.7 mm
- net 3.3V-4: track 0.65 -> 0.15 mm
Other:
- board text removed: "embrasse moi bordel"
- board text removed: "je rigole je t m"
- board text removed: "mon amour je t'aime énormément t'es trop sexy quand tu me parles de ton taf même si je capte R je t'aime"
