File: Amplificateur_Audio/Amplificateur_Audio_Custom/Channel_Generic.kicad_sch (KiCad schematic)
At the start: 81 parts, among them J401 SL+, J402 SL-, J403 SR+, J404 SR-, U401 PCM5252RHBR, U402 TPA3244DDWR, U403 74LVC1G125, U404 74LVC1G125

Commit message: Refactor : hierarchical template channels for multichannel routing
Parts:
- renumbered C410 to C?, C425 to C?, C431 to C?, C413 to C?, C409 to C?, C417 to C?, C401 to C?, C405 to C?, C426 to C?, C408 to C?, C412 to C?, C407 to C?, C445 to C?, C428 to C?, C437 to C?, C411 to C?, C402 to C?, C440 to C?, C403 to C?, C434 to C?, C444 to C?, C447 to C?, C446 to C?, C420 to C?, C427 to C?, C406 to C?, C423 to C?, C421 to C?, C435 to C?, C429 to C?, C416 to C?, C432 to C?, C439 to C?, C414 to C?, C438 to C?, C442 to C?, C443 to C?, C441 to C?, C404 to C?, C424 to C?, C418 to C?, C448 to C?, C419 to C?, C433 to C?, C430 to C?, C436 to C?, C415 to C?, C422 to C?, J403 to J?, J401 to J?, J404 to J?, J402 to J?, L402 to L?, L403 to L?, L401 to L?, R422 to R?, R408 to R?, R407 to R?, R413 to R?, R417 to R?, R412 to R?, R403 to R?, R415 to R?, R419 to R?, R406 to R?, R402 to R?, R411 to R?, R416 to R?, R420 to R?, R410 to R?, R421 to R?, R401 to R?, R405 to R?, R409 to R?, R404 to R?, R414 to R?, R418 to R?, U403 to U?, U402 to U?, U404 to U?, U401 to U?
Connections:
- net ADR2: no longer names the net of R?.1, R?.2, U?.22 (GPIO2/ADR2/GPO)
- net AVDD: no longer names the net of C?.2, C?.2, R?.1, U?.14 (AVDD)
- net BCK1 renamed BCK
- net CAPM: no longer names the net of C?.2, U?.8 (CAPM)
- net CAPP: no longer names the net of C?.1, U?.6 (CAPP)
- net DAC1L+ renamed DACL+
- net DAC1L- renamed DACL-
- net DAC1R+ renamed DACR+
- net DAC1R- renamed DACR-
- net DACF1L+ renamed DACFL+
- net DACF1L- renamed DACFL-
- net DACF1R+ renamed DACFR+
- net DACF1R- renamed DACFR-
- net DIN1 renamed DIN
- net INPUTL1+ renamed INPUTL+
- net INPUTL1- renamed INPUTL-
- net INPUTR1+ renamed INPUTR+
- net INPUTR1- renamed INPUTR-
- net LDOO: no longer names the net of C?.1, U?.2 (LDOO)
- net LRCK1 renamed LRCK
- net MISO: no longer names the net of R?.1, R?.2, U?.32 (MISO(GPIO1)/ADR1/FMT)
- net MODE1: no longer names the net of R?.2, U?.23 (MODE1)
- net MODE2: no longer names the net of R?.2, U?.24 (MS/MODE2)
- net OUT1A: no longer names the net of C?.1, L?.4, U?.27 (OUT_A), U?.28 (OUT_A)
- net OUT1B: no longer names the net of C?.1, L?.1, U?.32 (OUT_B)
- net OUT1C: no longer names the net of C?.1, L?.4, U?.35 (OUT_C)
- net OUT1D: no longer names the net of C?.1, L?.1, U?.39 (OUT_D), U?.40 (OUT_D)
- net OUTL1+: no longer names the net of R?.2, U?.10 (OUTLP)
- net OUTL1-: no longer names the net of R?.2, U?.11 (OUTLN)
- net OUTR1+: no longer names the net of R?.2, U?.13 (OUTRP)
- net OUTR1-: no longer names the net of R?.2, U?.12 (OUTRN)
- net SCK1 renamed SCK
- net SCL1 renamed SCL
- net SDA1 renamed SDA
- net Surrond Left+: no longer names the net of C?.2, C?.2, J?.1 (Pin_1), L?.3
- net Surrond Left-: no longer names the net of C?.2, C?.2, J?.1 (Pin_1), L?.2
- net Surrond Right+: no longer names the net of C?.2, C?.2, J?.1 (Pin_1), L?.3
- net SurroundRight-: no longer names the net of C?.2, C?.2, J?.1 (Pin_1), L?.2
- net VDD1: no longer names the net of C?.2, L?.2, U?.21 (VDD)
- net VNEG: no longer names the net of C?.1, U?.9 (VNEG)
- net XSMT: no longer names the net of R?.2, U?.1 (XSMT)
- net /AMP-RESET1 renamed /AMP-RESET
- net /CLIP_OTW1 renamed /CLIP_OTW
- net /FAULT1 renamed /FAULT
