File: Amplificateur_Audio/Amplificateur_Audio_Custom/Front_Right_Channel.kicad_sch (KiCad schematic)
At the start: 78 parts, among them J601 Front Right Tweeter+, J602 Front Right Tweeter-, J603 Front Right Woofer+, J604 Front Right Woofer-, U601 PCM5252RHBR, U602 TPA3244DDWR

Commit message: Assignation des composants et empreintes terminé
Parts:
- C601, C602, C605, C616, C617, C618, C619, C620, C621, C622, C623, C624, C625, C632, C633, C634, C635, C636, C641, C642, C643, C644: footprint (none) -> Capacitor_SMD:C_0603_1608Metric_Pad1.08x0.95mm_HandSolder
- C603, C604, C606, C607, C608, C609, C610, C611: footprint (none) -> Capacitor_SMD:C_0402_1005Metric_Pad0.74x0.62mm_HandSolder
- C612, C613, C614, C615, C626, C627, C628, C629, C630, C631: footprint (none) -> Capacitor_SMD:C_1206_3216Metric_Pad1.33x1.80mm_HandSolder
- C637, C638, C639, C640: footprint (none) -> Capacitor_SMD:C_1210_3225Metric_Pad1.33x2.70mm_HandSolder
- J601, J602, J603, J604: footprint (none) -> NewLibrary:630661MouserReel
- JP601, JP602, JP603, JP604: footprint (none) -> Connector_PinHeader_2.54mm:PinHeader_1x03_P2.54mm_Vertical_SMD_Pin1Left
- L601: footprint (none) -> Inductor_SMD:L_0603_1608Metric_Pad1.05x0.95mm_HandSolder
- L602, L603: footprint (none) -> NewLibrary:UA8014ALD
- R601, R609, R610, R611, R612, R613, R614, R615, R616, R617, R618, R619, R620, R621: footprint (none) -> Resistor_SMD:R_0603_1608Metric_Pad0.98x0.95mm_HandSolder
- R602, R605: value 4.99k -> 10k; footprint (none) -> Resistor_SMD:R_0402_1005Metric_Pad0.72x0.64mm_HandSolder; now not fitted
- R603: footprint (none) -> Resistor_SMD:R_0402_1005Metric_Pad0.72x0.64mm_HandSolder; now fitted
- R604: value 10k -> 4.99k; footprint (none) -> Resistor_SMD:R_0402_1005Metric_Pad0.72x0.64mm_HandSolder
- R606, R608: footprint (none) -> Resistor_SMD:R_0402_1005Metric_Pad0.72x0.64mm_HandSolder
- R607: value 10k -> 4.99k; footprint (none) -> Resistor_SMD:R_0402_1005Metric_Pad0.72x0.64mm_HandSolder; now fitted
- U601: footprint (none) -> Package_DFN_QFN:Texas_RHB0032E_VQFN-32-1EP_5x5mm_P0.5mm_EP3.45x3.45mm_ThermalVias
Connections:
- net 3.3V-4: now also C602.2, C604.2, R602.2, R605.2, R607.1, R608.2; no longer C601.2, C603.2, R603.2, R605.1, R606.1, R607.2
- net GND: now also C608.1, C625.2, R603.1, R606.1; no longer C608.2, C625.1, R602.1, R608.1
- net at R606.2: now also R605.1, U601.22 (GPIO2/ADR2/GPO); no longer U601.1 (XSMT)
- net at U602.9 (AVDD): now also C625.1; no longer C625.2
- net at R601.1, U601.14 (AVDD): now also C601.2, C603.2; no longer C602.2, C604.2
- net at U601.2 (LDOO): now also C608.2; no longer C608.1
- net at U601.23 (MODE1): now also R604.2; no longer R602.2
- net at U601.24 (MS/MODE2): now also R607.2; no longer R605.2
- new net: R608.1, U601.1 (XSMT)
- new net: R602.1, R603.2, U601.32 (MISO(GPIO1)/ADR1/FMT)

Commit message: Ajout de point de test et début du routage
Parts:
- C630, C631: footprint Capacitor_SMD:C_1206_3216Metric_Pad1.33x1.80mm_HandSolder -> Capacitor_SMD:CP_Elec_16x17.5
- U602: footprint DDV0044D_N -> NewLibrary:DDV0044D_N
Changed lines of the file:
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@@
 	)
 	(symbol
-		(lib_id "Device:C_Polarized_Small_US")
-		(at 276.225 68.58 0)
-		(unit 1)
-		(exclude_from_sim no)
-		(in_bom yes)
-		(on_board yes)
-		(dnp no)
-		(fields_autoplaced yes)
-		(property "Reference" "C630"
-			(at 278.765 66.8781 0)
-			(effects
-				(font
-					(size 1.27 1.27)
-				)
-				(justify left)
-			)
-		)
-		(property "Value" "1000uF"
-			(at 278.765 69.4181 0)
-			(effects
-				(font
-					(size 1.27 1.27)
-				)
-				(justify left)
-			)
-		)
-		(property "Footprint" "Capacitor_SMD:C_1206_3216Metric_Pad1.33x1.80mm_HandSolder"
-			(at 276.225 68.58 0)
-			(effects
-				(font
-					(size 1.27 1.27)
-				)
-				(hide yes)
-			)
-		)
-		(property "Datasheet" "~"
-			(at 276.225 68.58 0)
-			(effects
-				(font
-					(size 1.27 1.27)
-				)
-				(hide yes)
-			)
-		)
-		(property "Description" "GRM31MR71H105KA88L"
-			(at 276.225 68.58 0)
-			(effects
-				(font
-					(size 1.27 1.27)
-				)
-				(hide yes)
-			)
-		)
-		(pin "1"
-		)
-		(pin "2"
-		)
-		(instances
-			(project "Amplificateur_Audio"
-				(path "/bf9cc67f-178f-4c8c-b6a6-249a1896d599/cf8131f5-674c-4a4a-95bd-85b86419f228"
-					(reference "C630")
-					(unit 1)
-				)
-			)
-		)
-	)
-	(symbol
 		(lib_id "Device:C_Small")
 		(at 358.775 133.35 180)
@@
 			)
 		)
-		(property "Footprint" "DDV0044D_N"
+		(property "Footprint" "NewLibrary:DDV0044D_N"
 			(at 281.305 176.53 0)
 			(effects
@@
 	)
 	(symbol
+		(lib_id "Device:C_Polarized_Small_US")
+		(at 276.225 68.58 0)
+		(unit 1)
+		(exclude_from_sim no)
+		(in_bom yes)
+		(on_board yes)
+		(dnp no)
+		(fields_autoplaced yes)
+		(property "Reference" "C630"
+			(at 278.765 66.8781 0)
+			(effects
+				(font
+					(size 1.27 1.27)
+				)
+				(justify left)
+			)
+		)
+		(property "Value" "1000uF"
+			(at 278.765 69.4181 0)
+			(effects
+				(font
+					(size 1.27 1.27)
+				)
+				(justify left)
+			)
+		)
+		(property "Footprint" "Capacitor_SMD:CP_Elec_16x17.5"
+			(at 276.225 68.58 0)
+			(effects
+				(font
+					(size 1.27 1.27)
+				)
+				(hide yes)
+			)
+		)
+		(property "Datasheet" "~"
+			(at 276.225 68.58 0)
+			(effects
+				(font
+					(size 1.27 1.27)
+				)
+				(hide yes)
+			)
+		)
+		(property "Description" "EEV-FK1H102M"
+			(at 276.225 68.58 0)
+			(effects
+				(font
+					(size 1.27 1.27)
+				)
+				(hide yes)
+			)
+		)
+		(pin "1"
+		)
+		(pin "2"
+		)
+		(instances
+			(project "Amplificateur_Audio"
+				(path "/bf9cc67f-178f-4c8c-b6a6-249a1896d599/cf8131f5-674c-4a4a-95bd-85b86419f228"
+					(reference "C630")
+					(unit 1)
+				)
+			)
+		)
+	)
+	(symbol
 		(lib_id "Device:C_Small")
 		(at 258.445 68.58 180)
@@
 	)
 	(symbol
+		(lib_id "Device:C_Polarized_Small_US")
+		(at 282.575 87.63 0)
+		(unit 1)
+		(exclude_from_sim no)
+		(in_bom yes)
+		(on_board yes)
+		(dnp no)
+		(fields_autoplaced yes)
+		(property "Reference" "C631"
+			(at 285.115 85.9281 0)
+			(effects
+				(font
+					(size 1.27 1.27)
+				)
+				(justify left)
+			)
+		)
+		(property "Value" "1000uF"
+			(at 285.115 88.4681 0)
+			(effects
+				(font
+					(size 1.27 1.27)
+				)
+				(justify left)
+			)
+		)
+		(property "Footprint" "Capacitor_SMD:CP_Elec_16x17.5"
+			(at 282.575 87.63 0)
+			(effects
+				(font
+					(size 1.27 1.27)
+				)
+				(hide yes)
+			)
+		)
+		(property "Datasheet" "~"
+			(at 282.575 87.63 0)
+			(effects
+				(font
+					(size 1.27 1.27)
+				)
+				(hide yes)
+			)
+		)
+		(property "Description" "EEV-FK1H102M"
+			(at 282.575 87.63 0)
+			(effects
+				(font
+					(size 1.27 1.27)
+				)
+				(hide yes)
+			)
+		)
+		(pin "1"
+		)
+		(pin "2"
+		)
+		(instances
+			(project "Amplificateur_Audio"
+				(path "/bf9cc67f-178f-4c8c-b6a6-249a1896d599/cf8131f5-674c-4a4a-95bd-85b86419f228"
+					(reference "C631")
+					(unit 1)
+				)
+			)
+		)
+	)
+	(symbol
 		(lib_id "power:Earth")
 		(at 358.775 138.43 0)
@@
 					(unit 1)
 				)
-			)
-		)
-	)
-	(symbol
-		(lib_id "Device:C_Polarized_Small_US")
-		(at 282.575 87.63 0)
-		(unit 1)
-		(exclude_from_sim no)
-		(in_bom yes)
-		(on_board yes)
-		(dnp no)
-		(fields_autoplaced yes)
-		(property "Reference" "C631"
-			(at 285.115 85.9281 0)
-			(effects
-				(font
-					(size 1.27 1.27)
-				)
-				(justify left)
-			)
-		)
-		(property "Value" "1000uF"
-			(at 285.115 88.4681 0)
-			(effects
-				(font
-					(size 1.27 1.27)
-				)
-				(justify left)
-			)
-		)
-		(property "Footprint" "Capacitor_SMD:C_1206_3216Metric_Pad1.33x1.80mm_HandSolder"
-			(at 282.575 87.63 0)
-			(effects
-				(font
-					(size 1.27 1.27)
-				)
-				(hide yes)
-			)
-		)
-		(property "Datasheet" "~"
-			(at 282.575 87.63 0)
-			(effects
-				(font
-					(size 1.27 1.27)
-				)
-				(hide yes)
-			)
-		)
-		(property "Description" "GRM31MR71H105KA88L"
-			(at 282.575 87.63 0)
-			(effects
-				(font
-					(size 1.27 1.27)
-				)
-				(hide yes)
-			)
-		)
-		(pin "1"
-		)
-		(pin "2"
-		)
-		(instances
-			(project "Amplificateur_Audio"
-				(path "/bf9cc67f-178f-4c8c-b6a6-249a1896d599/cf8131f5-674c-4a4a-95bd-85b86419f228"
-					(reference "C631")
-					(unit 1)
-				)

Commit message: Refactor : hierarchical template channels for multichannel routing
Parts:
- removed JP601, JP602, JP603, JP604: Jumper_3_Open, Connector_PinHeader_2.54mm:PinHeader_1x03_P2.54mm_Vertical_SMD_Pin1Left, symbol Jumper:Jumper_3_Open
- added C624, C627: 0.1uF, Capacitor_SMD:C_0603_1608Metric, symbol Device:C_Small
- C601, C602, C605, C616, C617, C618, C619, C620, C621, C622, C623: footprint Capacitor_SMD:C_0603_1608Metric_Pad1.08x0.95mm_HandSolder -> Capacitor_SMD:C_0603_1608Metric
- C603, C604, C606, C609, C610, C611: footprint Capacitor_SMD:C_0402_1005Metric_Pad0.74x0.62mm_HandSolder -> Capacitor_SMD:C_0402_1005Metric
- C607: renamed from C608; footprint Capacitor_SMD:C_0402_1005Metric_Pad0.74x0.62mm_HandSolder -> Capacitor_SMD:C_0402_1005Metric
- C608: renamed from C607; footprint Capacitor_SMD:C_0402_1005Metric_Pad0.74x0.62mm_HandSolder -> Capacitor_SMD:C_0402_1005Metric
- C612, C613, C614, C615: footprint Capacitor_SMD:C_1206_3216Metric_Pad1.33x1.80mm_HandSolder -> Capacitor_SMD:C_1206_3216Metric
- C625: renamed from C624; footprint Capacitor_SMD:C_0603_1608Metric_Pad1.08x0.95mm_HandSolder -> Capacitor_SMD:C_0603_1608Metric
- C626: renamed from C625; footprint Capacitor_SMD:C_0603_1608Metric_Pad1.08x0.95mm_HandSolder -> Capacitor_SMD:C_0603_1608Metric
- C628: renamed from C626; footprint Capacitor_SMD:C_1206_3216Metric_Pad1.33x1.80mm_HandSolder -> Capacitor_SMD:C_1206_3216Metric
- C629: renamed from C627; footprint Capacitor_SMD:C_1206_3216Metric_Pad1.33x1.80mm_HandSolder -> Capacitor_SMD:C_1206_3216Metric
- C630: renamed from C628; footprint Capacitor_SMD:C_1206_3216Metric_Pad1.33x1.80mm_HandSolder -> Capacitor_SMD:C_1206_3216Metric
- C631: renamed from C629; footprint Capacitor_SMD:C_1206_3216Metric_Pad1.33x1.80mm_HandSolder -> Capacitor_SMD:C_1206_3216Metric
- C632: renamed from C630; footprint Capacitor_SMD:CP_Elec_16x17.5 -> NewLibrary:CAP_EEVFK1H102M
- C633: renamed from C631; footprint Capacitor_SMD:CP_Elec_16x17.5 -> NewLibrary:CAP_EEVFK1H102M
- C634: renamed from C632; footprint Capacitor_SMD:C_0603_1608Metric_Pad1.08x0.95mm_HandSolder -> Capacitor_SMD:C_0603_1608Metric
- C635: renamed from C633; footprint Capacitor_SMD:C_0603_1608Metric_Pad1.08x0.95mm_HandSolder -> Capacitor_SMD:C_0603_1608Metric
- C636: renamed from C634; footprint Capacitor_SMD:C_0603_1608Metric_Pad1.08x0.95mm_HandSolder -> Capacitor_SMD:C_0603_1608Metric
- C637: renamed from C635; footprint Capacitor_SMD:C_0603_1608Metric_Pad1.08x0.95mm_HandSolder -> Capacitor_SMD:C_0603_1608Metric
- C638: renamed from C636; footprint Capacitor_SMD:C_0603_1608Metric_Pad1.08x0.95mm_HandSolder -> Capacitor_SMD:C_0603_1608Metric
- C639: renamed from C637; footprint Capacitor_SMD:C_1210_3225Metric_Pad1.33x2.70mm_HandSolder -> Capacitor_SMD:C_1210_3225Metric
- C640: renamed from C638; footprint Capacitor_SMD:C_1210_3225Metric_Pad1.33x2.70mm_HandSolder -> Capacitor_SMD:C_1210_3225Metric
- C641: renamed from C639; footprint Capacitor_SMD:C_1210_3225Metric_Pad1.33x2.70mm_HandSolder -> Capacitor_SMD:C_1210_3225Metric
- C642: renamed from C640; footprint Capacitor_SMD:C_1210_3225Metric_Pad1.33x2.70mm_HandSolder -> Capacitor_SMD:C_1210_3225Metric
- C643: renamed from C641; footprint Capacitor_SMD:C_0603_1608Metric_Pad1.08x0.95mm_HandSolder -> Capacitor_SMD:C_0603_1608Metric
- C644: renamed from C642; footprint Capacitor_SMD:C_0603_1608Metric_Pad1.08x0.95mm_HandSolder -> Capacitor_SMD:C_0603_1608Metric
- C645: renamed from C643; footprint Capacitor_SMD:C_0603_1608Metric_Pad1.08x0.95mm_HandSolder -> Capacitor_SMD:C_0603_1608Metric
- C646: renamed from C644; footprint Capacitor_SMD:C_0603_1608Metric_Pad1.08x0.95mm_HandSolder -> Capacitor_SMD:C_0603_1608Metric
- R601, R613, R614, R615, R616, R617: footprint Resistor_SMD:R_0603_1608Metric_Pad0.98x0.95mm_HandSolder -> Resistor_SMD:R_0603_1608Metric
- R602, R603, R604, R605, R606, R607, R608: footprint Resistor_SMD:R_0402_1005Metric_Pad0.72x0.64mm_HandSolder -> Resistor_SMD:R_0402_1005Metric
Connections:
- net DAC3L+: now also C612.1
- net DAC3L-: now also C613.1
- net DAC3R+: now also C615.1
- net DAC3R-: now also C614.1
- net GND: now also C624.1, C627.1
- net PVDD: now also C624.2, C627.2
- net DACF3L+: now reaches C612.2, R613.2
- net AVDD: now reaches C601.2, C603.2, R601.1, U601.14 (AVDD)
- net VNEG: now reaches C609.1, U601.9 (VNEG)
- net DACF3L-: now reaches C613.2, R614.2
- net DACF3R+: now reaches C615.2, R616.2
- net DACF3R-: now reaches C614.2, R615.2
- net ADR2: now reaches R605.1, R606.2, U601.22 (GPIO2/ADR2/GPO)
- net XSMT: now reaches R608.1, U601.1 (XSMT)
- net MODE2: now reaches R607.2, U601.24 (MS/MODE2)
- net MODE1: now reaches R604.2, U601.23 (MODE1)
- net LDOO: now reaches C607.2, U601.2 (LDOO)
- net MISO: now reaches R602.1, R603.2, U601.32 (MISO(GPIO1)/ADR1/FMT)
- net CAPP: now reaches C608.1, U601.6 (CAPP)
- net CAPM: now reaches C608.2, U601.8 (CAPM)
- net INPUTA3 renamed INPUTL3+
- net INPUTB3 renamed INPUTL3-
- net INPUTC3 renamed INPUTR3-
- net INPUTD3 renamed INPUTR3+
- net OUTLN3 renamed OUTL3-
- net OUTLP3 renamed OUTL3+
- net OUTRN3 renamed OUTR3-
- net OUTRP3 renamed OUTR3+
Other:
- note removed: "FROM INPUT HEADER"
- moved on the sheet: C608, C620, C621, C622, C623, C625, C626, C628, C629, C630, C631, C632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
