File: Amplificateur_Audio/Amplificateur_Audio_Custom/Up_Channel.kicad_sch (KiCad schematic)
At the start: 78 parts, among them J502 UP LEFT+, J503 UP LEFT-, J504 UP RIGHT+, J505 UP RIGHT-, U501 PCM5252RHBR, U502 TPA3244DDWR

Commit message: Ajout de l'assignation des compostants et des empreintes jusqu'à la page 6
Parts:
- removed C529: 1uF, symbol Device:C_Small
- removed C533: 1000uF, symbol Device:C_Polarized_Small_US
- removed C545, C546: 0.01uF, symbol Device:C_Small
- removed R522: 3.3, symbol Device:R_Small
- added C501, C503: 10uF, Capacitor_SMD:C_0603_1608Metric_Pad1.08x0.95mm_HandSolder, symbol Device:C_Small
- added C529: 1000uF, Capacitor_SMD:C_1206_3216Metric_Pad1.33x1.80mm_HandSolder, symbol Device:C_Polarized_Small_US
- added C533: 0.033uF, Capacitor_SMD:C_0603_1608Metric_Pad1.08x0.95mm_HandSolder, symbol Device:C_Small
- added R518: 3.3, Resistor_SMD:R_0603_1608Metric_Pad0.98x0.95mm_HandSolder, symbol Device:R_Small
- C502, C518, C519, C522, C523, C534, C535, C536, C544: footprint (none) -> Capacitor_SMD:C_0603_1608Metric_Pad1.08x0.95mm_HandSolder
- C504, C507: value 10uF -> 0.1uF; footprint (none) -> Capacitor_SMD:C_0402_1005Metric_Pad0.74x0.62mm_HandSolder
- C505, C506, C509, C511: footprint (none) -> Capacitor_SMD:C_0402_1005Metric_Pad0.74x0.62mm_HandSolder
- C508, C510: value 0.1uF -> 1000pF; footprint (none) -> Capacitor_SMD:C_0402_1005Metric_Pad0.74x0.62mm_HandSolder
- C512, C513: value 1000pF -> 10uF; footprint (none) -> Capacitor_SMD:C_1206_3216Metric_Pad1.33x1.80mm_HandSolder
- C514, C515, C527, C528, C530, C531, C532: footprint (none) -> Capacitor_SMD:C_1206_3216Metric_Pad1.33x1.80mm_HandSolder
- C516, C517: value 10uF -> 100pF; footprint (none) -> Capacitor_SMD:C_0603_1608Metric_Pad1.08x0.95mm_HandSolder
- C520, C521: value 100pF -> 0.1uF; footprint (none) -> Capacitor_SMD:C_0603_1608Metric_Pad1.08x0.95mm_HandSolder
- C524: value 0.1uF -> 1uF; footprint (none) -> Capacitor_SMD:C_0603_1608Metric_Pad1.08x0.95mm_HandSolder
- C525: value 0.047uF -> 1uF; footprint (none) -> Capacitor_SMD:C_0603_1608Metric_Pad1.08x0.95mm_HandSolder
- C526: value 1uF -> 0.047uF; footprint (none) -> Capacitor_SMD:C_0603_1608Metric_Pad1.08x0.95mm_HandSolder
- C537: value 0.033uF -> 1uF; footprint (none) -> Capacitor_SMD:C_1210_3225Metric_Pad1.33x2.70mm_HandSolder
- C538: value 0.1uF -> 0.01uF; footprint (none) -> Capacitor_SMD:C_0603_1608Metric_Pad1.08x0.95mm_HandSolder
- C539, C541: footprint (none) -> Capacitor_SMD:C_1210_3225Metric_Pad1.33x2.70mm_HandSolder
- C540, C542: value 1uF -> 0.01uF; footprint (none) -> Capacitor_SMD:C_0603_1608Metric_Pad1.08x0.95mm_HandSolder
- C543: value 0.01uF -> 1uF; footprint (none) -> Capacitor_SMD:C_1210_3225Metric_Pad1.33x2.70mm_HandSolder
- J501: renamed from J502; footprint (none) -> NewLibrary:630661MouserReel
- J502: renamed from J503; footprint (none) -> NewLibrary:630661MouserReel
- J503: renamed from J504; footprint (none) -> NewLibrary:630661MouserReel
- J504: renamed from J505; footprint (none) -> NewLibrary:630661MouserReel
- JP501, JP502, JP503, JP504: footprint (none) -> Connector_PinHeader_2.54mm:PinHeader_1x03_P2.54mm_Vertical_SMD_Pin1Left
- L501: footprint (none) -> Inductor_SMD:L_0603_1608Metric_Pad1.05x0.95mm_HandSolder
- L502, L503: footprint (none) -> NewLibrary:UA8014ALD
- R501, R509, R510, R511, R512, R513, R514, R515, R516, R517, R519, R520, R521: footprint (none) -> Resistor_SMD:R_0603_1608Metric_Pad0.98x0.95mm_HandSolder
- R502, R503, R504, R505, R506, R507, R508: footprint (none) -> Resistor_SMD:R_0402_1005Metric_Pad0.72x0.64mm_HandSolder
- U501: footprint (none) -> Package_DFN_QFN:Texas_RHB0032E_VQFN-32-1EP_5x5mm_P0.5mm_EP3.45x3.45mm_ThermalVias
Connections:
- net 12V: now also C520.2, C522.2; no longer C523.2, C524.2
- net 3.3V-4: now also C504.2, R506.2, C501.2; no longer C507.2, C508.2, R506.1
- net DAC2L+: now also C508.1; no longer C512.1
- net DAC2L-: now also C508.2; no longer C512.2
- net DAC2R+: now also C510.2; no longer C513.2
- net DAC2R-: now also C510.1; no longer C513.1
- net DVDD2: now also C524.1; no longer C526.1
- net GND: now also C516.2, C517.2, C520.1, C521.1, C524.2, C525.2, C526.1, C537.1, C543.1, C501.1, C503.1, C529.2, R518.2; no longer C508.1, C510.2, C520.2, C521.2, C524.1, C525.1, C526.2, C538.1, C540.1, C542.1
- net INPUTA2: now also C516.1; no longer C518.1
- net INPUTB2: now also C517.1; no longer C519.1
- net INPUTC2: now also C518.1; no longer C520.1
- net INPUTD2: now also C519.1; no longer C521.1
- net OUT2A: now also C533.1; no longer C534.1
- net OUT2B: now also C534.1; no longer C536.1
- net OUT2D: now also C536.1; no longer C537.1
- net PVDD: now also C527.2, C529.1
- net UpL+: now also C537.2, C538.2; no longer C539.2, C543.2
- net UpL-: now also C539.2; no longer C544.2
- net UpR+: now also C542.2
- net UpR-: now also C543.2, C544.2; no longer C542.2
- net VDD2: now also C521.2; no longer C522.2
- net at C514.1: now also JP503.2 (C); no longer JP501.2 (C)
- net at R513.2: now also C512.2; no longer C514.2
- net at C506.2, R501.1, U501.14 (AVDD): now also C503.2; no longer C504.2
- net at R516.2: now also C515.2; no longer C517.2
- net at R519.1: now also C540.1; no longer C543.1
- net at U502.44 (BST_D): now also C536.2; no longer C537.2
- net at R515.2: now also C514.2; no longer C516.2
- net at U502.24 (BST_B): now also C534.2; no longer C536.2
- net at U502.3 (VBG): now also C523.2; no longer C538.2
- net at JP502.2 (C): now also C513.1; no longer C515.1
- net at U501.1 (XSMT): now also R506.1; no longer R506.2
- net at U502.8 (C_START): now also C526.2; no longer C525.2
- net at JP504.2 (C): now also C515.1; no longer C517.1
- net at R521.1: now also C544.1
- net at R514.2: now also C513.2; no longer C515.2
- net at U501.2 (LDOO): now also C507.2; no longer C510.1
- net at U502.9 (AVDD): now also C525.1; no longer C527.2
- net at U502.23 (BST_A): now also C533.2; no longer C534.2
- net at R520.1: now also C542.1; no longer C544.1
- new net: C538.1, R518.1
- new net: C512.1, JP501.2 (C)

Commit message: Ajout de point de test et début du routage
Parts:
- C529, C532: footprint Capacitor_SMD:C_1206_3216Metric_Pad1.33x1.80mm_HandSolder -> Capacitor_SMD:CP_Elec_16x17.5
- U502: footprint DDV0044D_N -> NewLibrary:DDV0044D_N

Commit message: Refactor : hierarchical template channels for multichannel routing
Parts:
- removed JP501, JP502, JP503, JP504: Jumper_3_Open, Connector_PinHeader_2.54mm:PinHeader_1x03_P2.54mm_Vertical_SMD_Pin1Left, symbol Jumper:Jumper_3_Open
- added C525, C527: 0.1uF, Capacitor_SMD:C_0603_1608Metric, symbol Device:C_Small
- C501: renamed from C503; footprint Capacitor_SMD:C_0603_1608Metric_Pad1.08x0.95mm_HandSolder -> Capacitor_SMD:C_0603_1608Metric
- C502: renamed from C501; footprint Capacitor_SMD:C_0603_1608Metric_Pad1.08x0.95mm_HandSolder -> Capacitor_SMD:C_0603_1608Metric
- C503: renamed from C506; footprint Capacitor_SMD:C_0402_1005Metric_Pad0.74x0.62mm_HandSolder -> Capacitor_SMD:C_0402_1005Metric
- C504: footprint Capacitor_SMD:C_0402_1005Metric_Pad0.74x0.62mm_HandSolder -> Capacitor_SMD:C_0402_1005Metric
- C505: renamed from C502; footprint Capacitor_SMD:C_0603_1608Metric_Pad1.08x0.95mm_HandSolder -> Capacitor_SMD:C_0603_1608Metric
- C506: renamed from C505; footprint Capacitor_SMD:C_0402_1005Metric_Pad0.74x0.62mm_HandSolder -> Capacitor_SMD:C_0402_1005Metric
- C507: renamed from C509; footprint Capacitor_SMD:C_0402_1005Metric_Pad0.74x0.62mm_HandSolder -> Capacitor_SMD:C_0402_1005Metric
- C508: renamed from C507; footprint Capacitor_SMD:C_0402_1005Metric_Pad0.74x0.62mm_HandSolder -> Capacitor_SMD:C_0402_1005Metric
- C509: renamed from C511; footprint Capacitor_SMD:C_0402_1005Metric_Pad0.74x0.62mm_HandSolder -> Capacitor_SMD:C_0402_1005Metric
- C510: renamed from C508; footprint Capacitor_SMD:C_0402_1005Metric_Pad0.74x0.62mm_HandSolder -> Capacitor_SMD:C_0402_1005Metric
- C511: renamed from C510; footprint Capacitor_SMD:C_0402_1005Metric_Pad0.74x0.62mm_HandSolder -> Capacitor_SMD:C_0402_1005Metric
- C512, C513, C514, C515, C531: footprint Capacitor_SMD:C_1206_3216Metric_Pad1.33x1.80mm_HandSolder -> Capacitor_SMD:C_1206_3216Metric
- C516, C517, C518, C519, C524, C535: footprint Capacitor_SMD:C_0603_1608Metric_Pad1.08x0.95mm_HandSolder -> Capacitor_SMD:C_0603_1608Metric
- C520: renamed from C521; footprint Capacitor_SMD:C_0603_1608Metric_Pad1.08x0.95mm_HandSolder -> Capacitor_SMD:C_0603_1608Metric
- C521: renamed from C522; footprint Capacitor_SMD:C_0603_1608Metric_Pad1.08x0.95mm_HandSolder -> Capacitor_SMD:C_0603_1608Metric
- C522: renamed from C520; footprint Capacitor_SMD:C_0603_1608Metric_Pad1.08x0.95mm_HandSolder -> Capacitor_SMD:C_0603_1608Metric
- C523: renamed from C526; footprint Capacitor_SMD:C_0603_1608Metric_Pad1.08x0.95mm_HandSolder -> Capacitor_SMD:C_0603_1608Metric
- C526: renamed from C525; footprint Capacitor_SMD:C_0603_1608Metric_Pad1.08x0.95mm_HandSolder -> Capacitor_SMD:C_0603_1608Metric
- C528: renamed from C527; footprint Capacitor_SMD:C_1206_3216Metric_Pad1.33x1.80mm_HandSolder -> Capacitor_SMD:C_1206_3216Metric
- C529: renamed from C530; footprint Capacitor_SMD:C_1206_3216Metric_Pad1.33x1.80mm_HandSolder -> Capacitor_SMD:C_1206_3216Metric
- C530: renamed from C528; footprint Capacitor_SMD:C_1206_3216Metric_Pad1.33x1.80mm_HandSolder -> Capacitor_SMD:C_1206_3216Metric
- C532: renamed from C529; footprint Capacitor_SMD:CP_Elec_16x17.5 -> NewLibrary:CAP_EEVFK1H102M
- C533: renamed from C532; footprint Capacitor_SMD:CP_Elec_16x17.5 -> NewLibrary:CAP_EEVFK1H102M
- C534: renamed from C533; footprint Capacitor_SMD:C_0603_1608Metric_Pad1.08x0.95mm_HandSolder -> Capacitor_SMD:C_0603_1608Metric
- C536: renamed from C534; footprint Capacitor_SMD:C_0603_1608Metric_Pad1.08x0.95mm_HandSolder -> Capacitor_SMD:C_0603_1608Metric
- C537: renamed from C536; footprint Capacitor_SMD:C_0603_1608Metric_Pad1.08x0.95mm_HandSolder -> Capacitor_SMD:C_0603_1608Metric
- C538: renamed from C523; footprint Capacitor_SMD:C_0603_1608Metric_Pad1.08x0.95mm_HandSolder -> Capacitor_SMD:C_0603_1608Metric
- C539: renamed from C537; footprint Capacitor_SMD:C_1210_3225Metric_Pad1.33x2.70mm_HandSolder -> Capacitor_SMD:C_1210_3225Metric
- C540: renamed from C539; footprint Capacitor_SMD:C_1210_3225Metric_Pad1.33x2.70mm_HandSolder -> Capacitor_SMD:C_1210_3225Metric
- C541: footprint Capacitor_SMD:C_1210_3225Metric_Pad1.33x2.70mm_HandSolder -> Capacitor_SMD:C_1210_3225Metric
- C542: renamed from C543; footprint Capacitor_SMD:C_1210_3225Metric_Pad1.33x2.70mm_HandSolder -> Capacitor_SMD:C_1210_3225Metric
- C543: renamed from C538; footprint Capacitor_SMD:C_0603_1608Metric_Pad1.08x0.95mm_HandSolder -> Capacitor_SMD:C_0603_1608Metric
- C544: renamed from C540; footprint Capacitor_SMD:C_0603_1608Metric_Pad1.08x0.95mm_HandSolder -> Capacitor_SMD:C_0603_1608Metric
- C545: renamed from C542; footprint Capacitor_SMD:C_0603_1608Metric_Pad1.08x0.95mm_HandSolder -> Capacitor_SMD:C_0603_1608Metric
- C546: renamed from C544; footprint Capacitor_SMD:C_0603_1608Metric_Pad1.08x0.95mm_HandSolder -> Capacitor_SMD:C_0603_1608Metric
- R501, R513, R514, R515, R516, R517: footprint Resistor_SMD:R_0603_1608Metric_Pad0.98x0.95mm_HandSolder -> Resistor_SMD:R_0603_1608Metric
- R502: renamed from R503; footprint Resistor_SMD:R_0402_1005Metric_Pad0.72x0.64mm_HandSolder -> Resistor_SMD:R_0402_1005Metric
- R503: renamed from R504; footprint Resistor_SMD:R_0402_1005Metric_Pad0.72x0.64mm_HandSolder -> Resistor_SMD:R_0402_1005Metric
- R504: renamed from R502; footprint Resistor_SMD:R_0402_1005Metric_Pad0.72x0.64mm_HandSolder -> Resistor_SMD:R_0402_1005Metric
- R505: renamed from R507; footprint Resistor_SMD:R_0402_1005Metric_Pad0.72x0.64mm_HandSolder -> Resistor_SMD:R_0402_1005Metric
- R506: renamed from R508; footprint Resistor_SMD:R_0402_1005Metric_Pad0.72x0.64mm_HandSolder -> Resistor_SMD:R_0402_1005Metric
- R507: renamed from R505; footprint Resistor_SMD:R_0402_1005Metric_Pad0.72x0.64mm_HandSolder -> Resistor_SMD:R_0402_1005Metric
- R508: renamed from R506; footprint Resistor_SMD:R_0402_1005Metric_Pad0.72x0.64mm_HandSolder -> Resistor_SMD:R_0402_1005Metric
Connections:
- net DAC2L+: now also C512.1
- net DAC2L-: now also C513.1
- net DAC2R+: now also C515.1
- net DAC2R-: now also C514.1
- net GND: now also C525.1, C527.1
- net PVDD: now also C525.2, C527.2
- net XSMT: now reaches R508.1, U501.1 (XSMT)
- net CAPP: now reaches C507.1, U501.6 (CAPP)
- net CAPM: now reaches C507.2, U501.8 (CAPM)
- net MODE2: now reaches R507.2, U501.24 (MS/MODE2)
- net DACF2R+: now reaches C515.2, R516.2
- net LDOO: now reaches C508.2, U501.2 (LDOO)
- net MODE1: now reaches R504.2, U501.23 (MODE1)
- net DACF2L-: now reaches C513.2, R514.2
- net MISO: now reaches R502.1, R503.2, U501.32 (MISO(GPIO1)/ADR1/FMT)
- net ADR2: now reaches R505.1, R506.2, U501.22 (GPIO2/ADR2/GPO)
- net DACF2L+: now reaches C512.2, R513.2
- net VNEG: now reaches C509.1, U501.9 (VNEG)
- net AVDD: now reaches C501.2, C503.2, R501.1, U501.14 (AVDD)
- net DACF2R-: now reaches C514.2, R515.2
- net INPUTA2 renamed INPUTL2+
- net INPUTB2 renamed INPUTL2-
- net INPUTC2 renamed INPUTR2-
- net INPUTD2 renamed INPUTR2+
- net OUTLN2 renamed OUTL2-
- net OUTLP2 renamed OUTL2+
- net OUTRN2 renamed OUTR2-
- net OUTRP2 renamed OUTR2+
Other:
- note removed: "FROM INPUT HEADER"
- moved on the sheet: C507
