File: Amplificateur_Audio/Amplificateur_Audio_Custom/Analog_Io_Board.kicad_sch (KiCad schematic)
At the start: 147 parts, among them J1101 SURROUND-LEFT, J1102 UPMIX-LEFT, J1103 FR-TWEETER, J1104 FL-TWEETER, J1105 CENTER-TWEETER, J1106 SURROUND-RIGHT, J1107 UPMIX-RIGHT, J1108 FR-WOOFER, J1109 FL-WOOFER, J1110 CENTER-WOOFER, J1111 Analog OUTPUT Connector, U1101 NE5532AD, U1102 NE5532AD, U1103 NE5532AD, U1104 NE5532AD, U1105 NE5532AD, U1106 NE5532AD, U1107 NE5532AD, U1108 NE5532AD, U1109 NE5532AD, U1110 NE5532AD

Commit message: Assignation des composants et empreintes terminé
Parts:
- C1101, C1106, C1110, C1114, C1118, C1122, C1126, C1130, C1134, C1138, C1142, C1144, C1146, C1148, C1150, C1152, C1154, C1156, C1158, C1160: footprint (none) -> Capacitor_SMD:C_0402_1005Metric_Pad0.74x0.62mm_HandSolder
- C1102, C1105, C1109, C1113, C1117, C1121, C1125, C1129, C1133, C1137: footprint (none) -> Capacitor_SMD:C_1206_3216Metric_Pad1.33x1.80mm_HandSolder
- C1103, C1104, C1107, C1108, C1111, C1112, C1115, C1116, C1119, C1120, C1123, C1124, C1127, C1128, C1131, C1132, C1135, C1136, C1139, C1140, C1163: footprint (none) -> Capacitor_SMD:C_0603_1608Metric_Pad1.08x0.95mm_HandSolder
- C1161, C1162: footprint (none) -> Capacitor_SMD:C_0805_2012Metric_Pad1.18x1.45mm_HandSolder
- C1165, C1167: value 0.1uF -> 10uF
- D1101: footprint (none) -> LED_SMD:LED_0805_2012Metric_Pad1.15x1.40mm_HandSolder
- FB1101, FB1102, R1101, R1102, R1103, R1104, R1105, R1106, R1107, R1108, R1109, R1110, R1111, R1112, R1113, R1114, R1115, R1116, R1117, R1118, R1119, R1120, R1121, R1122, R1123, R1124, R1125, R1126, R1127, R1128, R1129, R1130, R1131, R1132, R1133, R1134, R1135, R1136, R1137, R1138, R1139, R1140, R1141, R1142, R1143, R1144, R1145, R1146, R1147, R1148, R1149, R1150, R1151, R1152, R1153, R1154, R1155: footprint (none) -> Resistor_SMD:R_0402_1005Metric_Pad0.72x0.64mm_HandSolder
- J1101, J1102, J1103, J1104, J1105, J1106, J1107, J1108, J1109, J1110: footprint (none) -> NewLibrary:CUI_RCJ-024
- J1111: footprint (none) -> Connector_PinHeader_2.54mm:PinHeader_2x25_P2.54mm_Vertical_SMD
- L1101: footprint (none) -> Inductor_SMD:L_APV_ANR4012
- U1101, U1102, U1103, U1104, U1105, U1106, U1107, U1108, U1109, U1110: footprint (none) -> Package_SO:Texas_HTSOP-8-1EP_3.9x4.9mm_P1.27mm_EP2.95x4.9mm_Mask2.4x3.1mm_ThermalVias

Commit message: Ajout de point de test et début du routage
Parts:
- C1141, C1143, C1145, C1147, C1149, C1151, C1153, C1155, C1157, C1159, C1164, C1165, C1166, C1167: footprint (none) -> Capacitor_SMD:C_0603_1608Metric_Pad1.08x0.95mm_HandSolder
Changed lines of the file:
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@@
 			)
 		)
-		(property "Footprint" ""
+		(property "Footprint" "Capacitor_SMD:C_0603_1608Metric_Pad1.08x0.95mm_HandSolder"
 			(at 109.855 227.965 0)
 			(effects
@@
 			)
 		)
-		(property "Footprint" ""
+		(property "Footprint" "Capacitor_SMD:C_0603_1608Metric_Pad1.08x0.95mm_HandSolder"
 			(at 31.75 272.415 0)
 			(effects
@@
 			)
 		)
-		(property "Footprint" ""
+		(property "Footprint" "Capacitor_SMD:C_0603_1608Metric_Pad1.08x0.95mm_HandSolder"
 			(at 85.09 227.965 0)
 			(effects
@@
 			)
 		)
-		(property "Footprint" ""
+		(property "Footprint" "Capacitor_SMD:C_0603_1608Metric_Pad1.08x0.95mm_HandSolder"
 			(at 76.2 227.965 0)
 			(effects
@@
 			)
 		)
-		(property "Footprint" ""
+		(property "Footprint" "Capacitor_SMD:C_0603_1608Metric_Pad1.08x0.95mm_HandSolder"
 			(at 120.65 272.415 0)
 			(effects
@@
 			)
 		)
-		(property "Footprint" ""
+		(property "Footprint" "Capacitor_SMD:C_0603_1608Metric_Pad1.08x0.95mm_HandSolder"
 			(at 53.34 272.415 0)
 			(effects
@@
 			)
 		)
-		(property "Footprint" ""
+		(property "Footprint" "Capacitor_SMD:C_0603_1608Metric_Pad1.08x0.95mm_HandSolder"
 			(at 74.93 272.415 0)
 			(effects
@@
 			)
 		)
-		(property "Footprint" ""
+		(property "Footprint" "Capacitor_SMD:C_0603_1608Metric_Pad1.08x0.95mm_HandSolder"
 			(at 53.34 249.555 0)
 			(effects
@@
 			)
 		)
-		(property "Footprint" ""
+		(property "Footprint" "Capacitor_SMD:C_0603_1608Metric_Pad1.08x0.95mm_HandSolder"
 			(at 31.75 249.555 0)
 			(effects
@@
 			)
 		)
-		(property "Footprint" ""
+		(property "Footprint" "Capacitor_SMD:C_0603_1608Metric_Pad1.08x0.95mm_HandSolder"
 			(at 74.93 249.555 0)
 			(effects
@@
 			)
 		)
-		(property "Footprint" ""
+		(property "Footprint" "Capacitor_SMD:C_0603_1608Metric_Pad1.08x0.95mm_HandSolder"
 			(at 97.79 272.415 0)
 			(effects
@@
 			)
 		)
-		(property "Footprint" ""
+		(property "Footprint" "Capacitor_SMD:C_0603_1608Metric_Pad1.08x0.95mm_HandSolder"
 			(at 97.79 249.555 0)
 			(effects
@@
 			)
 		)
-		(property "Footprint" ""
+		(property "Footprint" "Capacitor_SMD:C_0603_1608Metric_Pad1.08x0.95mm_HandSolder"
 			(at 120.65 249.555 0)
 			(effects
@@
 			)
 		)
-		(property "Footprint" ""
+		(property "Footprint" "Capacitor_SMD:C_0603_1608Metric_Pad1.08x0.95mm_HandSolder"
 			(at 118.745 227.965 0)
 			(effects

Commit message: Refactor : hierarchical template channels for multichannel routing
Parts:
- C1101, C1106, C1110, C1114, C1118, C1122, C1126, C1130, C1134, C1138, C1142, C1144, C1146, C1148, C1150, C1152, C1154, C1156, C1158, C1160: footprint Capacitor_SMD:C_0402_1005Metric_Pad0.74x0.62mm_HandSolder -> Capacitor_SMD:C_0402_1005Metric
- C1102, C1105, C1109, C1113, C1117, C1121, C1125, C1129, C1133, C1137: footprint Capacitor_SMD:C_1206_3216Metric_Pad1.33x1.80mm_HandSolder -> Capacitor_SMD:C_1206_3216Metric
- C1103, C1104, C1107, C1108, C1111, C1112, C1115, C1116, C1119, C1120, C1123, C1124, C1127, C1128, C1131, C1132, C1135, C1136, C1139, C1140, C1141, C1143, C1145, C1147, C1149, C1151, C1153, C1155, C1157, C1159, C1163, C1164, C1165, C1166, C1167: footprint Capacitor_SMD:C_0603_1608Metric_Pad1.08x0.95mm_HandSolder -> Capacitor_SMD:C_0603_1608Metric
- C1161, C1162: footprint Capacitor_SMD:C_0805_2012Metric_Pad1.18x1.45mm_HandSolder -> Capacitor_SMD:C_0805_2012Metric
